File: mark-II-Rpi-devkit/KiCAD/SJ201-Raspberry Pi 4 Daughterboard/RaspberryPi.sch (KiCad schematic (older format))
At the start: 65 parts, among them J6 Raspberry_Pi_4, J7 USB_B_Micro, J9 USB_A, P1 LED, P2 LED, P3 LED, P4 LED, SW1 MuteMic, U6 FE1.1s, Y2 12MHz

Commit message: Update BOM
Parts:
- J6: footprint user:PinSocket_2x20_P2.54mm_RightAngle_SMD -> Connector_PinSocket_2.54mm:PinSocket_2x20_P2.54mm_Horizontal; Description (none) -> 2X20 PIN 2.54MM DOUBLE ROW RIGHT ANGLE FEMALE PIN HEADER; Digikey 609-5967-ND -> (none); Link (none) -> https://www.taydaelectronics.com/connectors-sockets/2x20-pi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; MPN 71609-320LF -> FH412-2*20P 0.8U
Changed lines of the file:
@@
 Sheet 5 6
 Title "Raspberry Pi"
-Date "2020-07-10"
-Rev "0.59"
+Date "2020-07-14"
+Rev "0.60"
 Comp "Mycroft"
 Comment1 "MCU Connections"
@@
 F 0 "J6" H 2150 4156 50  0000 C CNN
 F 1 "Raspberry_Pi_4" H 2895 4110 50  0000 C CNN
-F 2 "user:PinSocket_2x20_P2.54mm_RightAngle_SMD" H 2150 2675 50  0001 C CNN
+F 2 "Connector_PinSocket_2.54mm:PinSocket_2x20_P2.54mm_Horizontal" H 2150 2675 50  0001 C CNN
 F 3 "https://www.raspberrypi.org/documentation/hardware/raspberrypi/schematics/rpi_SCH_3bplus_1p0_reduced.pdf" H 2150 2675 50  0001 C CNN
-F 4 "609-5967-ND" H 2150 2675 50  0001 C CNN "Digikey"
-F 5 "71609-320LF" H 2150 2675 50  0001 C CNN "MPN"
+F 4 "FH412-2*20P 0.8U" H 2150 2675 50  0001 C CNN "MPN"
+F 5 "2X20 PIN 2.54MM DOUBLE ROW RIGHT ANGLE FEMALE PIN HEADER" H 2150 2675 50  0001 C CNN "Description"
+F 6 "https://www.taydaelectronics.com/connectors-sockets/2x20-pin-2-54mm-dounle-row-right-angle-female-pin-header.html" H 2150 2675 50  0001 C CNN "Link"
 	1    2150 2675
 	1    0    0    -1

Commit message: Update BOM - fix OPL numbers for Seeed PCBA
Parts:
- ACT1, P1, P2, P3, P4: Link (none) -> https://lcsc.com/product-detail/Others_TOGIALED-TJ-S1608SW6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; MPN TJ-S1608SW6TGLC2R-A5 -> 19-217-R6C-AL1M2VY-3T; SKU (none) -> 304090042
- D10, D11, D12, D13, D2, D3, D4, D5, D6, D7, D8, D9: Link (none) -> https://lcsc.com/product-detail/Others_WS2813-Mini-WS2813-3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
Changed lines of the file:
@@
 F 3 "https://datasheet.lcsc.com/szlcsc/1810010024_Worldsemi-WS2813-Mini-WS2813-3535_C189639.pdf" H 1675 5200 50  0001 L TNN
 F 4 "WS2813-MINI(WS2813-3535)" H 1575 5575 50  0001 C CNN "MPN"
+F 5 "https://lcsc.com/product-detail/Others_WS2813-Mini-WS2813-3535_C189639.html" H 1575 5575 50  0001 C CNN "Link"
 	1    1575 5575
 	1    0    0    -1
@@
 F 3 "https://datasheet.lcsc.com/szlcsc/1810010024_Worldsemi-WS2813-Mini-WS2813-3535_C189639.pdf" H 2375 5200 50  0001 L TNN
 F 4 "WS2813-MINI(WS2813-3535)" H 2275 5575 50  0001 C CNN "MPN"
+F 5 "https://lcsc.com/product-detail/Others_WS2813-Mini-WS2813-3535_C189639.html" H 2275 5575 50  0001 C CNN "Link"
 	1    2275 5575
 	1    0    0    -1
@@
 F 3 "https://datasheet.lcsc.com/szlcsc/1810010024_Worldsemi-WS2813-Mini-WS2813-3535_C189639.pdf" H 3125 5200 50  0001 L TNN
 F 4 "WS2813-MINI(WS2813-3535)" H 3025 5575 50  0001 C CNN "MPN"
+F 5 "https://lcsc.com/product-detail/Others_WS2813-Mini-WS2813-3535_C189639.html" H 3025 5575 50  0001 C CNN "Link"
 	1    3025 5575
 	1    0    0    -1
@@
 F 3 "https://datasheet.lcsc.com/szlcsc/1810010024_Worldsemi-WS2813-Mini-WS2813-3535_C189639.pdf" H 3850 5200 50  0001 L TNN
 F 4 "WS2813-MINI(WS2813-3535)" H 3750 5575 50  0001 C CNN "MPN"
+F 5 "https://lcsc.com/product-detail/Others_WS2813-Mini-WS2813-3535_C189639.html" H 3750 5575 50  0001 C CNN "Link"
 	1    3750 5575
 	1    0    0    -1
@@
 F 3 "https://datasheet.lcsc.com/szlcsc/1810010024_Worldsemi-WS2813-Mini-WS2813-3535_C189639.pdf" H 4600 5200 50  0001 L TNN
 F 4 "WS2813-MINI(WS2813-3535)" H 4500 5575 50  0001 C CNN "MPN"
+F 5 "https://lcsc.com/product-detail/Others_WS2813-Mini-WS2813-3535_C189639.html" H 4500 5575 50  0001 C CNN "Link"
 	1    4500 5575
 	1    0    0    -1
@@
 F 3 "https://datasheet.lcsc.com/szlcsc/1810010024_Worldsemi-WS2813-Mini-WS2813-3535_C189639.pdf" H 5300 5200 50  0001 L TNN
 F 4 "WS2813-MINI(WS2813-3535)" H 5200 5575 50  0001 C CNN "MPN"
+F 5 "https://lcsc.com/product-detail/Others_WS2813-Mini-WS2813-3535_C189639.html" H 5200 5575 50  0001 C CNN "Link"
 	1    5200 5575
 	1    0    0    -1
@@
 F 3 "https://datasheet.lcsc.com/szlcsc/1810010024_Worldsemi-WS2813-Mini-WS2813-3535_C189639.pdf" H 6050 5200 50  0001 L TNN
 F 4 "WS2813-MINI(WS2813-3535)" H 5950 5575 50  0001 C CNN "MPN"
+F 5 "https://lcsc.com/product-detail/Others_WS2813-Mini-WS2813-3535_C189639.html" H 5950 5575 50  0001 C CNN "Link"
+F 6 "https://lcsc.com/product-detail/Others_WS2813-Mini-WS2813-3535_C189639.html" H 5950 5575 50  0001 C CNN "Link"
 	1    5950 5575
 	1    0    0    -1
@@
 F 3 "https://datasheet.lcsc.com/szlcsc/1810010024_Worldsemi-WS2813-Mini-WS2813-3535_C189639.pdf" H 6775 5200 50  0001 L TNN
 F 4 "WS2813-MINI(WS2813-3535)" H 6675 5575 50  0001 C CNN "MPN"
+F 5 "https://lcsc.com/product-detail/Others_WS2813-Mini-WS2813-3535_C189639.html" H 6675 5575 50  0001 C CNN "Link"
 	1    6675 5575
 	1    0    0    -1
@@
 F 3 "https://datasheet.lcsc.com/szlcsc/1810010024_Worldsemi-WS2813-Mini-WS2813-3535_C189639.pdf" H 7475 5200 50  0001 L TNN
 F 4 "WS2813-MINI(WS2813-3535)" H 7375 5575 50  0001 C CNN "MPN"
+F 5 "https://lcsc.com/product-detail/Others_WS2813-Mini-WS2813-3535_C189639.html" H 7375 5575 50  0001 C CNN "Link"
 	1    7375 5575
 	1    0    0    -1
@@
 F 3 "https://datasheet.lcsc.com/szlcsc/1810010024_Worldsemi-WS2813-Mini-WS2813-3535_C189639.pdf" H 8150 5200 50  0001 L TNN
 F 4 "WS2813-MINI(WS2813-3535)" H 8050 5575 50  0001 C CNN "MPN"
+F 5 "https://lcsc.com/product-detail/Others_WS2813-Mini-WS2813-3535_C189639.html" H 8050 5575 50  0001 C CNN "Link"
+F 6 "https://lcsc.com/product-detail/Others_WS2813-Mini-WS2813-3535_C189639.html" H 8050 5575 50  0001 C CNN "Link"
 	1    8050 5575
 	1    0    0    -1
@@
 F 3 "https://datasheet.lcsc.com/szlcsc/1810010024_Worldsemi-WS2813-Mini-WS2813-3535_C189639.pdf" H 9550 5200 50  0001 L TNN
 F 4 "WS2813-MINI(WS2813-3535)" H 9450 5575 50  0001 C CNN "MPN"
+F 5 "https://lcsc.com/product-detail/Others_WS2813-Mini-WS2813-3535_C189639.html" H 9450 5575 50  0001 C CNN "Link"
 	1    9450 5575
 	1    0    0    -1
@@
 F 3 "https://datasheet.lcsc.com/szlcsc/1810010024_Worldsemi-WS2813-Mini-WS2813-3535_C189639.pdf" H 8850 5200 50  0001 L TNN
 F 4 "WS2813-MINI(WS2813-3535)" H 8750 5575 50  0001 C CNN "MPN"
+F 5 "https://lcsc.com/product-detail/Others_WS2813-Mini-WS2813-3535_C189639.html" H 8750 5575 50  0001 C CNN "Link"
 	1    8750 5575
 	1    0    0    -1
@@
 F 2 "LED_SMD:LED_0603_1608Metric" H 8850 3675 50  0001 C CNN
 F 3 "https://datasheet.lcsc.com/szlcsc/1811141223_TOGIALED-TJ-S1608SW6TGLC2R-A5_C192315.pdf" H 8850 3675 50  0001 C CNN
-F 4 "TJ-S1608SW6TGLC2R-A5" H 8850 3675 50  0001 C CNN "MPN"
+F 4 "19-217-R6C-AL1M2VY-3T" H 8850 3675 50  0001 C CNN "MPN"
 F 5 "C192315" H 8850 3675 50  0001 C CNN "LCSC"
+F 6 "https://lcsc.com/product-detail/Others_TOGIALED-TJ-S1608SW6TGLC2R-A5_C192315.html" H 8850 3675 50  0001 C CNN "Link"
+F 7 "304090042" H 8850 3675 50  0001 C CNN "SKU"
 	1    8850 3675
 	1    0    0    -1
@@
 F 2 "LED_SMD:LED_0603_1608Metric" H 8850 3825 50  0001 C CNN
 F 3 "https://datasheet.lcsc.com/szlcsc/1811141223_TOGIALED-TJ-S1608SW6TGLC2R-A5_C192315.pdf" H 8850 3825 50  0001 C CNN
-F 4 "TJ-S1608SW6TGLC2R-A5" H 8850 3825 50  0001 C CNN "MPN"
+F 4 "19-217-R6C-AL1M2VY-3T" H 8850 3825 50  0001 C CNN "MPN"
 F 5 "C192315" H 8850 3825 50  0001 C CNN "LCSC"
+F 6 "https://lcsc.com/product-detail/Others_TOGIALED-TJ-S1608SW6TGLC2R-A5_C192315.html" H 8850 3825 50  0001 C CNN "Link"
+F 7 "304090042" H 8850 3825 50  0001 C CNN "SKU"
 	1    8850 3825
 	-1   0    0    1
@@
 F 2 "LED_SMD:LED_0603_1608Metric" H 9225 4450 50  0001 C CNN
 F 3 "https://datasheet.lcsc.com/szlcsc/1811141223_TOGIALED-TJ-S1608SW6TGLC2R-A5_C192315.pdf" H 9225 4450 50  0001 C CNN
-F 4 "TJ-S1608SW6TGLC2R-A5" H 9225 4450 50  0001 C CNN "MPN"
+F 4 "19-217-R6C-AL1M2VY-3T" H 9225 4450 50  0001 C CNN "MPN"
 F 5 "C192315" H 9225 4450 50  0001 C CNN "LCSC"
+F 6 "https://lcsc.com/product-detail/Others_TOGIALED-TJ-S1608SW6TGLC2R-A5_C192315.html" H 9225 4450 50  0001 C CNN "Link"
+F 7 "304090042" H 9225 4450 50  0001 C CNN "SKU"
 	1    9225 4450
 	0    -1   -1   0
@@
 F 2 "LED_SMD:LED_0603_1608Metric" H 8850 4125 50  0001 C CNN
 F 3 "https://datasheet.lcsc.com/szlcsc/1811141223_TOGIALED-TJ-S1608SW6TGLC2R-A5_C192315.pdf" H 8850 4125 50  0001 C CNN
-F 4 "TJ-S1608SW6TGLC2R-A5" H 8850 4125 50  0001 C CNN "MPN"
+F 4 "19-217-R6C-AL1M2VY-3T" H 8850 4125 50  0001 C CNN "MPN"
 F 5 "C192315" H 8850 4125 50  0001 C CNN "LCSC"
+F 6 "https://lcsc.com/product-detail/Others_TOGIALED-TJ-S1608SW6TGLC2R-A5_C192315.html" H 8850 4125 50  0001 C CNN "Link"
+F 7 "304090042" H 8850 4125 50  0001 C CNN "SKU"
 	1    8850 4125
 	1    0    0    -1
@@
 F 2 "LED_SMD:LED_0603_1608Metric" H 8850 4275 50  0001 C CNN
 F 3 "https://datasheet.lcsc.com/szlcsc/1811141223_TOGIALED-TJ-S1608SW6TGLC2R-A5_C192315.pdf" H 8850 4275 50  0001 C CNN
-F 4 "TJ-S1608SW6TGLC2R-A5" H 8850 4275 50  0001 C CNN "MPN"
+F 4 "19-217-R6C-AL1M2VY-3T" H 8850 4275 50  0001 C CNN "MPN"
 F 5 "C192315" H 8850 4275 50  0001 C CNN "LCSC"
+F 6 "https://lcsc.com/product-detail/Others_TOGIALED-TJ-S1608SW6TGLC2R-A5_C192315.html" H 8850 4275 50  0001 C CNN "Link"
+F 7 "304090042" H 8850 4275 50  0001 C CNN "SKU"
 	1    8850 4275
 	-1   0    0    1

Commit message: Updated KiCAD files to 0.63 for PCB printing & Assembly at JLCPCB
Parts:
- removed J9: USB_A, Connector_USB:USB_A_Wuerth_614004134726_Horizontal, symbol Connector:USB_A
- added DM3, DP3: TestPoint, TestPoint:TestPoint_Pad_D1.0mm, symbol Connector:TestPoint
- ACT1, P1, P2, P3, P4: LCSC C192315 -> C72043
- C28, C29, C31, C33: LCSC (none) -> C1525
- C30, C32, C34: LCSC (none) -> C15525
- D1: LCSC (none) -> C2128
- R23: LCSC (none) -> C25792
- R29, R33, R38: LCSC (none) -> C25104
- R30: LCSC (none) -> C25741
- R31: footprint Resistor_SMD:R_0402_1005Metric -> Resistor_SMD:R_0603_1608Metric; LCSC (none) -> C13167; MPN 0402WGF2701TCE -> RTT032701FTP
Connections:
- wire segments 178 -> 175
Changed lines of the file:
@@
 Sheet 5 6
 Title "Raspberry Pi"
-Date "2020-07-14"
-Rev "0.60"
+Date "2020-07-22"
+Rev "0.63"
 Comp "Mycroft"
 Comment1 "MCU Connections"
@@
 F 0 "R31" H 6459 4246 50  0000 L CNN
 F 1 "2.7k" H 6459 4155 50  0000 L CNN
-F 2 "Resistor_SMD:R_0402_1005Metric" H 6400 4200 50  0001 C CNN
+F 2 "Resistor_SMD:R_0603_1608Metric" H 6400 4200 50  0001 C CNN
 F 3 "~" H 6400 4200 50  0001 C CNN
-F 4 "0402WGF2701TCE" H 6400 4200 50  0001 C CNN "MPN"
+F 4 "RTT032701FTP" H 6400 4200 50  0001 C CNN "MPN"
+F 5 "C13167" H 6400 4200 50  0001 C CNN "LCSC"
 	1    6400 4200
 	1    0    0    -1
@@
 F 3 "~" H 5825 2775 50  0001 C CNN
 F 4 "0402WGF1003TCE" H 5825 2775 50  0001 C CNN "MPN"
+F 5 "C25741" H 5825 2775 50  0001 C CNN "LCSC"
 	1    5825 2775
 	1    0    0    -1
@@
 	1    0    0    -1
 $EndComp
-$Comp
-L Connector:USB_A J9
-U 1 1 5F3ACA75
-P 9425 3250
-F 0 "J9" H 9195 3239 50  0000 R CNN
-F 1 "USB_A" H 9195 3148 50  0000 R CNN
-F 2 "Connector_USB:USB_A_Wuerth_614004134726_Horizontal" H 9575 3200 50  0001 C CNN
-F 3 " ~" H 9575 3200 50  0001 C CNN
-	1    9425 3250
-	-1   0    0    -1
-$EndComp
 Wire Wire Line
 	8425 3250 8425 2875
@@
 Wire Wire Line
 	8350 2975 8350 3350
-$Comp
-L power:GND #PWR062
-U 1 1 5F3B2C33
-P 9425 3650
-F 0 "#PWR062" H 9425 3400 50  0001 C CNN
-F 1 "GND" H 9430 3477 50  0000 C CNN
-F 2 "" H 9425 3650 50  0001 C CNN
-F 3 "" H 9425 3650 50  0001 C CNN
-	1    9425 3650
-	1    0    0    -1
-$EndComp
-Wire Wire Line
-	9525 3650 9425 3650
-Connection ~ 9425 3650
 Wire Wire Line
 	8425 3250 9125 3250
@@
 F 4 "CC0402MRX5R5BB106" H 8180 1825 20  0001 C CNN "MPN"
 F 5 "302010053" V 8066 1607 20  0001 R CNN "SKU"
+F 6 "C15525" H 8150 1675 50  0001 C CNN "LCSC"
 	1    8150 1675
 	0    -1   -1   0
@@
 F 4 "CC0402MRX5R5BB106" H 7130 1825 20  0001 C CNN "MPN"
 F 5 "302010053" V 7016 1607 20  0001 R CNN "SKU"
+F 6 "C15525" H 7100 1675 50  0001 C CNN "LCSC"
 	1    7100 1675
 	0    -1   -1   0
@@
 F 4 "CC0402MRX5R5BB106" H 6430 1825 20  0001 C CNN "MPN"
 F 5 "302010053" V 6316 1607 20  0001 R CNN "SKU"
+F 6 "C15525" H 6400 1675 50  0001 C CNN "LCSC"
 	1    6400 1675
 	0    -1   -1   0
@@
 F 4 "CC0402KRX7R8BB104" H 6130 1825 20  0001 C CNN "MPN"
 F 5 "302010024" H 6130 1825 20  0001 C CNN "SKU"
+F 6 "C1525" H 6100 1675 50  0001 C CNN "LCSC"
 	1    6100 1675
 	0    1    1    0
@@
 F 4 "CC0402KRX7R8BB104" H 6830 1825 20  0001 C CNN "MPN"
 F 5 "302010024" H 6830 1825 20  0001 C CNN "SKU"
+F 6 "C1525" H 6800 1675 50  0001 C CNN "LCSC"
 	1    6800 1675
 	0    1    1    0
@@
 F 4 "CC0402KRX7R8BB104" H 7780 1825 20  0001 C CNN "MPN"
 F 5 "302010024" H 7780 1825 20  0001 C CNN "SKU"
+F 6 "C1525" H 7750 1675 50  0001 C CNN "LCSC"
 	1    7750 1675
 	0    1    1    0
@@
 F 3 "~" H 1050 4850 50  0001 C CNN
 F 4 "1N4148WSF-7" H 1050 4850 50  0001 C CNN "MPN"
+F 5 "C2128" H 1050 4850 50  0001 C CNN "LCSC"
 	1    1050 4850
 	-1   0    0    1
@@
 F 4 "CC0402KRX7R8BB104" H 1330 5150 20  0001 C CNN "MPN"
 F 5 "302010024" H 1330 5150 20  0001 C CNN "SKU"
+F 6 "C1525" H 1300 5000 50  0001 C CNN "LCSC"
 	1    1300 5000
 	0    1    1    0
@@
 	1    0    0    -1
 $EndComp
-$Comp
-L power:+5V #PWR?
-U 1 1 5F0EF0E6
-P 9000 3025
-AR Path="/5EAAC9A5/5F0EF0E6" Ref="#PWR?"  Part="1"
-AR Path="/5EA9C461/5F0EF0E6" Ref="#PWR0120"  Part="1"
-F 0 "#PWR0120" H 9000 2875 50  0001 C CNN
-F 1 "+5V" H 9000 3175 50  0000 C CNN
-F 2 "" H 9000 3025 50  0001 C CNN
-F 3 "" H 9000 3025 50  0001 C CNN
-	1    9000 3025
-	1    0    0    -1
-$EndComp
-Wire Wire Line
-	9125 3050 9000 3050
-Wire Wire Line
-	9000 3050 9000 3025
 $Comp
 L power:+5V #PWR?
@@
 F 4 "RC0402JR-0747KL" H 5825 2175 50  0001 C CNN "MPN"
 F 5 "301010005" H 5825 2175 50  0001 C CNN "SKU"
+F 6 "C25792" H 5825 2175 50  0001 C CNN "LCSC"
 	1    5825 2175
 	-1   0    0    1
@@
 F 3 "https://datasheet.lcsc.com/szlcsc/1811141223_TOGIALED-TJ-S1608SW6TGLC2R-A5_C192315.pdf" H 8850 3675 50  0001 C CNN
 F 4 "19-217-R6C-AL1M2VY-3T" H 8850 3675 50  0001 C CNN "MPN"
-F 5 "C192315" H 8850 3675 50  0001 C CNN "LCSC"
+F 5 "C72043" H 8850 3675 50  0001 C CNN "LCSC"
 F 6 "https://lcsc.com/product-detail/Others_TOGIALED-TJ-S1608SW6TGLC2R-A5_C192315.html" H 8850 3675 50  0001 C CNN "Link"
 F 7 "304090042" H 8850 3675 50  0001 C CNN "SKU"
@@
 F 3 "~" H 8325 3675 50  0001 C CNN
 F 4 "0402WGF3300TCE" H 8325 3675 50  0001 C CNN "MPN"
+F 5 "C25104" H 8325 3675 50  0001 C CNN "LCSC"
 	1    8325 3675
 	0    -1   -1   0
@@
 F 3 "https://datasheet.lcsc.com/szlcsc/1811141223_TOGIALED-TJ-S1608SW6TGLC2R-A5_C192315.pdf" H 8850 3825 50  0001 C CNN
 F 4 "19-217-R6C-AL1M2VY-3T" H 8850 3825 50  0001 C CNN "MPN"
-F 5 "C192315" H 8850 3825 50  0001 C CNN "LCSC"
+F 5 "C72043" H 8850 3825 50  0001 C CNN "LCSC"
 F 6 "https://lcsc.com/product-detail/Others_TOGIALED-TJ-S1608SW6TGLC2R-A5_C192315.html" H 8850 3825 50  0001 C CNN "Link"
 F 7 "304090042" H 8850 3825 50  0001 C CNN "SKU"
@@
 F 3 "~" H 8325 3775 50  0001 C CNN
 F 4 "0402WGF3300TCE" H 8325 3775 50  0001 C CNN "MPN"
+F 5 "C25104" H 8325 3775 50  0001 C CNN "LCSC"
 	1    8325 3775
 	0    -1   -1   0
@@
 F 3 "https://datasheet.lcsc.com/szlcsc/1811141223_TOGIALED-TJ-S1608SW6TGLC2R-A5_C192315.pdf" H 9225 4450 50  0001 C CNN
 F 4 "19-217-R6C-AL1M2VY-3T" H 9225 4450 50  0001 C CNN "MPN"
-F 5 "C192315" H 9225 4450 50  0001 C CNN "LCSC"
+F 5 "C72043" H 9225 4450 50  0001 C CNN "LCSC"
 F 6 "https://lcsc.com/product-detail/Others_TOGIALED-TJ-S1608SW6TGLC2R-A5_C192315.html" H 9225 4450 50  0001 C CNN "Link"
 F 7 "304090042" H 9225 4450 50  0001 C CNN "SKU"
@@
 F 3 "~" H 9225 4700 50  0001 C CNN
 F 4 "0402WGF3300TCE" H 9225 4700 50  0001 C CNN "MPN"
+F 5 "C25104" H 9225 4700 50  0001 C CNN "LCSC"
 	1    9225 4700
 	-1   0    0    1
@@
 F 3 "https://datasheet.lcsc.com/szlcsc/1811141223_TOGIALED-TJ-S1608SW6TGLC2R-A5_C192315.pdf" H 8850 4125 50  0001 C CNN
 F 4 "19-217-R6C-AL1M2VY-3T" H 8850 4125 50  0001 C CNN "MPN"
-F 5 "C192315" H 8850 4125 50  0001 C CNN "LCSC"
+F 5 "C72043" H 8850 4125 50  0001 C CNN "LCSC"
 F 6 "https://lcsc.com/product-detail/Others_TOGIALED-TJ-S1608SW6TGLC2R-A5_C192315.html" H 8850 4125 50  0001 C CNN "Link"
 F 7 "304090042" H 8850 4125 50  0001 C CNN "SKU"
@@
 F 3 "https://datasheet.lcsc.com/szlcsc/1811141223_TOGIALED-TJ-S1608SW6TGLC2R-A5_C192315.pdf" H 8850 4275 50  0001 C CNN
 F 4 "19-217-R6C-AL1M2VY-3T" H 8850 4275 50  0001 C CNN "MPN"
-F 5 "C192315" H 8850 4275 50  0001 C CNN "LCSC"
+F 5 "C72043" H 8850 4275 50  0001 C CNN "LCSC"
 F 6 "https://lcsc.com/product-detail/Others_TOGIALED-TJ-S1608SW6TGLC2R-A5_C192315.html" H 8850 4275 50  0001 C CNN "Link"
 F 7 "304090042" H 8850 4275 50  0001 C CNN "SKU"
@@
 Wire Wire Line
 	3300 2325 3300 2400
+$Comp
+L Connector:TestPoint DP3
+U 1 1 5F505183
+P 9125 3250
+F 0 "DP3" V 9125 3600 50  0000 R CNN
+F 1 "TestPoint" V 9125 4000 50  0001 R CNN
+F 2 "TestPoint:TestPoint_Pad_D1.0mm" H 9325 3250 50  0001 C CNN
+F 3 "~" H 9325 3250 50  0001 C CNN
+	1    9125 3250
+	0    1    1    0
+$EndComp
+$Comp
+L Connector:TestPoint DM3
+U 1 1 5F5056AD
+P 9125 3350
+F 0 "DM3" V 9125 3700 50  0000 R CNN
+F 1 "TestPoint" V 9125 4100 50  0001 R CNN
+F 2 "TestPoint:TestPoint_Pad_D1.0mm" H 9325 3350 50  0001 C CNN
+F 3 "~" H 9325 3350 50  0001 C CNN
+	1    9125 3350
+	0    1    1    0
+$EndComp
 $EndSCHEMATC

Commit message: Change USB IC to CM108B, add in Line Out jack, prep for 2 PCB sandwich
Parts:
- D10, D11, D12, D13, D3, D4, D5, D6, D7, D8, D9: value WS2813 -> WS2812B; footprint user:LED_WS2813_3.5x3.5mm_P1.1mm -> user:LED_WS2812_Mini_3.5x3.5mm_P1.1mm; symbol LED:WS2813 -> LED:WS2812B; LCSC (none) -> C114583; Link https://lcsc.com/product-detail/Others_WS2813-Mini-WS2813-3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 -> https://lcsc.com/product-detail/Others_WS2812B-Mini-WS2812B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; MPN WS2813-MINI(WS2813-3535) -> WS2812B-MINI(WS2812B-3535)
- D2: value WS2813 -> WS2812B; footprint user:LED_WS2813_3.5x3.5mm_P1.1mm -> user:LED_WS2812_Mini_3.5x3.5mm_P1.1mm; symbol LED:WS2813 -> LED:WS2812B; LCSC (none) -> C114583; Link https://lcsc.com/product-detail/Others_WS2813-Mini-WS2813-3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 -> (none); MPN WS2813-MINI(WS2813-3535) -> WS2812B-Mini
- S1, S2, S3: LCSC (none) -> C318884
Connections:
- wire segments 175 -> 124
- no-connect marks 9 -> 8

Commit message: Mark 2 - PCB Files to the printer
Parts:
- J7: LCSC (none) -> C319162
- SW1: LCSC (none) -> C221841
Changed lines of the file:
@@
 F 4 "2073-USB3076-30-ATR-ND" H 4525 2475 50  0001 C CNN "Digikey"
 F 5 "U254-051T-4BH83-F1B" H 4525 2475 50  0001 C CNN "MPN"
+F 6 "C319162" H 4525 2475 50  0001 C CNN "LCSC"
 	1    4525 2475
 	1    0    0    -1
@@
 F 4 "PCM12SMTR" H 5125 6775 50  0001 C CNN "MPN"
 F 5 "401-2016-2-ND" H 5125 6775 50  0001 C CNN "Digikey"
+F 6 "C221841" H 5125 6775 50  0001 C CNN "LCSC"
 	1    5125 6775
 	1    0    0    -1

Commit message: Update to v0.66 - printed at JLC - 2nd spin
Parts:
- TP18: footprint TestPoint:TestPoint_Pad_D1.0mm -> TestPoint:TestPoint_Pad_D2.0mm
- Y2: symbol Device:Crystal_GND23 -> Device:Crystal_GND24
Changed lines of the file:
@@
 Sheet 5 6
 Title "Raspberry Pi"
-Date "2020-07-24"
-Rev "0.65"
+Date "2020-08-16"
+Rev "0.66"
 Comp "Mycroft"
 Comment1 "MCU Connections"
@@
 F 0 "TP18" H 1175 6150 50  0000 R CNN
 F 1 "TestPoint" H 1175 6225 50  0000 R CNN
-F 2 "TestPoint:TestPoint_Pad_D1.0mm" H 1425 6100 50  0001 C CNN
+F 2 "TestPoint:TestPoint_Pad_D2.0mm" H 1425 6100 50  0001 C CNN
 F 3 "~" H 1425 6100 50  0001 C CNN
 	1    1225 6100
@@
 $EndComp
 $Comp
-L Device:Crystal_GND23 Y2
+L Device:Crystal_GND24 Y2
 U 1 1 5F963155
 P 5825 3825
