File: mark-II-Rpi-devkit/KiCAD/SJ201-Raspberry Pi 4 Daughterboard/RaspberryPi.sch (KiCad schematic (older format))
At the start: 66 parts, among them J6 Raspberry_Pi_4, J7 USB_B_Micro, P1 LED, P2 LED, P3 LED, P4 LED, SW1 MuteMic, U6 FE1.1s, Y2 12MHz

Commit message: Fix missing items in schematic in Github
Parts:
- C28, C29, C31, C33: symbol OPL_Capacitor:CERAMIC-100NF-50V-10%-X7R_0805_ -> Device:C_Small
- C30, C32, C34: symbol OPL_Capacitor:CERAMIC-2.2UF-25V-10%-X7R_0805_ -> Device:C_Small
Connections:
- wire segments 124 -> 138
Changed lines of the file:
@@
 Wire Wire Line
 	7650 1975 7650 2075
-Wire Wire Line
-	7650 1975 7650 1525
 Connection ~ 7650 1975
 $Comp
@@
 NoConn ~ 8050 3275
 $Comp
-L OPL_Capacitor:CERAMIC-2.2UF-25V-10%-X7R_0805_ C?
+L Device:C_Small C?
 U 1 1 5EEEBC4D
 P 8150 1675
 AR Path="/5EA9C76D/5EEEBC4D" Ref="C?"  Part="1"
 AR Path="/5EA9C461/5EEEBC4D" Ref="C34"  Part="1"
-F 0 "C34" V 8192 1607 45  0000 R CNN
-F 1 "10UF" V 8108 1607 45  0000 R CNN
+F 0 "C34" H 8100 1600 45  0000 R CNN
+F 1 "10UF" H 8100 1750 45  0000 R CNN
 F 2 "Capacitor_SMD:C_0402_1005Metric" H 8150 1675 50  0001 C CNN
 F 3 "" H 8150 1675 50  0001 C CNN
@@
 F 6 "C15525" H 8150 1675 50  0001 C CNN "LCSC"
 	1    8150 1675
-	0    -1   -1   0
-$EndComp
-$Comp
-L OPL_Capacitor:CERAMIC-2.2UF-25V-10%-X7R_0805_ C?
+	-1   0    0    1
+$EndComp
+$Comp
+L Device:C_Small C?
 U 1 1 5EEEEE5E
 P 7100 1675
 AR Path="/5EA9C76D/5EEEEE5E" Ref="C?"  Part="1"
 AR Path="/5EA9C461/5EEEEE5E" Ref="C32"  Part="1"
-F 0 "C32" V 7142 1607 45  0000 R CNN
-F 1 "10UF" V 7058 1607 45  0000 R CNN
+F 0 "C32" H 7050 1600 45  0000 R CNN
+F 1 "10UF" H 7050 1750 45  0000 R CNN
 F 2 "Capacitor_SMD:C_0402_1005Metric" H 7100 1675 50  0001 C CNN
 F 3 "" H 7100 1675 50  0001 C CNN
@@
 F 6 "C15525" H 7100 1675 50  0001 C CNN "LCSC"
 	1    7100 1675
-	0    -1   -1   0
-$EndComp
-Connection ~ 7100 1525
-Wire Wire Line
-	7100 1525 7350 1525
-$Comp
-L OPL_Capacitor:CERAMIC-2.2UF-25V-10%-X7R_0805_ C?
+	-1   0    0    1
+$EndComp
+$Comp
+L Device:C_Small C?
 U 1 1 5EEEF2E1
 P 6400 1675
 AR Path="/5EA9C76D/5EEEF2E1" Ref="C?"  Part="1"
 AR Path="/5EA9C461/5EEEF2E1" Ref="C30"  Part="1"
-F 0 "C30" V 6442 1607 45  0000 R CNN
-F 1 "10UF" V 6358 1607 45  0000 R CNN
+F 0 "C30" H 6350 1600 45  0000 R CNN
+F 1 "10UF" H 6350 1750 45  0000 R CNN
 F 2 "Capacitor_SMD:C_0402_1005Metric" H 6400 1675 50  0001 C CNN
 F 3 "" H 6400 1675 50  0001 C CNN
@@
 F 6 "C15525" H 6400 1675 50  0001 C CNN "LCSC"
 	1    6400 1675
-	0    -1   -1   0
-$EndComp
-$Comp
-L OPL_Capacitor:CERAMIC-100NF-50V-10%-X7R_0805_ C?
+	-1   0    0    1
+$EndComp
+$Comp
+L Device:C_Small C?
 U 1 1 5EF91B9F
 P 6100 1675
 AR Path="/5EA9C76D/5EF91B9F" Ref="C?"  Part="1"
 AR Path="/5EA9C461/5EF91B9F" Ref="C29"  Part="1"
-F 0 "C29" V 6058 1743 45  0000 L CNN
-F 1 "100NF" V 6142 1743 45  0000 L CNN
+F 0 "C29" H 6150 1750 45  0000 L CNN
+F 1 "100NF" H 6150 1600 45  0000 L CNN
 F 2 "Capacitor_SMD:C_0402_1005Metric" H 6100 1675 50  0001 C CNN
 F 3 "" H 6100 1675 50  0001 C CNN
@@
 F 6 "C1525" H 6100 1675 50  0001 C CNN "LCSC"
 	1    6100 1675
-	0    1    1    0
-$EndComp
-Wire Wire Line
-	6025 1525 6100 1525
-Connection ~ 6100 1525
-Wire Wire Line
-	6100 1525 6400 1525
-$Comp
-L OPL_Capacitor:CERAMIC-100NF-50V-10%-X7R_0805_ C?
+	1    0    0    -1
+$EndComp
+$Comp
+L Device:C_Small C?
 U 1 1 5EF964F8
 P 6800 1675
 AR Path="/5EA9C76D/5EF964F8" Ref="C?"  Part="1"
 AR Path="/5EA9C461/5EF964F8" Ref="C31"  Part="1"
-F 0 "C31" V 6758 1743 45  0000 L CNN
-F 1 "100NF" V 6850 1725 45  0000 L CNN
+F 0 "C31" H 6850 1750 45  0000 L CNN
+F 1 "100NF" H 6850 1600 45  0000 L CNN
 F 2 "Capacitor_SMD:C_0402_1005Metric" H 6800 1675 50  0001 C CNN
 F 3 "" H 6800 1675 50  0001 C CNN
@@
 F 6 "C1525" H 6800 1675 50  0001 C CNN "LCSC"
 	1    6800 1675
-	0    1    1    0
-$EndComp
-Wire Wire Line
-	6800 1525 7100 1525
-Wire Wire Line
-	7650 1525 7750 1525
-$Comp
-L OPL_Capacitor:CERAMIC-100NF-50V-10%-X7R_0805_ C?
+	1    0    0    -1
+$EndComp
+$Comp
+L Device:C_Small C?
 U 1 1 5EF9B304
 P 7750 1675
 AR Path="/5EA9C76D/5EF9B304" Ref="C?"  Part="1"
 AR Path="/5EA9C461/5EF9B304" Ref="C33"  Part="1"
-F 0 "C33" V 7708 1743 45  0000 L CNN
-F 1 "100NF" V 7792 1743 45  0000 L CNN
+F 0 "C33" H 7800 1750 45  0000 L CNN
+F 1 "100NF" H 7800 1600 45  0000 L CNN
 F 2 "Capacitor_SMD:C_0402_1005Metric" H 7750 1675 50  0001 C CNN
 F 3 "" H 7750 1675 50  0001 C CNN
@@
 F 6 "C1525" H 7750 1675 50  0001 C CNN "LCSC"
 	1    7750 1675
-	0    1    1    0
-$EndComp
-Connection ~ 7750 1525
-Wire Wire Line
-	7750 1525 8150 1525
+	1    0    0    -1
+$EndComp
 $Comp
 L power:GND #PWR0101
@@
 	1225 5575 1200 5575
 $Comp
-L OPL_Capacitor:CERAMIC-100NF-50V-10%-X7R_0805_ C?
+L Device:C_Small C?
 U 1 1 5EEF814C
 P 1300 5000
 AR Path="/5EA9C76D/5EEF814C" Ref="C?"  Part="1"
 AR Path="/5EA9C461/5EEF814C" Ref="C28"  Part="1"
-F 0 "C28" V 1258 5068 45  0000 L CNN
-F 1 "100NF" V 1375 5050 45  0000 L CNN
+F 0 "C28" H 1350 5075 45  0000 L CNN
+F 1 "100NF" H 1350 4925 45  0000 L CNN
 F 2 "Capacitor_SMD:C_0402_1005Metric" H 1300 5000 50  0001 C CNN
 F 3 "" H 1300 5000 50  0001 C CNN
@@
 F 6 "C1525" H 1300 5000 50  0001 C CNN "LCSC"
 	1    1300 5000
-	0    1    1    0
+	1    0    0    -1
 $EndComp
 $Comp
@@
 $EndComp
 Wire Wire Line
-	1300 4850 1200 4850
-Wire Wire Line
-	1300 4850 1575 4850
-Wire Wire Line
 	1575 4850 1575 5275
-Connection ~ 1300 4850
 Text Notes 775  4700 0    51   ~ 0
 Drop first LED voltage to \n4.3v with Diode
@@
 Wire Wire Line
 	6975 5575 7075 5575
+Wire Wire Line
+	1200 4850 1300 4850
+Wire Wire Line
+	1300 4900 1300 4850
+Connection ~ 1300 4850
+Wire Wire Line
+	1300 4850 1575 4850
+Wire Wire Line
+	1300 5100 1300 5150
+Wire Wire Line
+	6800 1525 7100 1525
+Wire Wire Line
+	6025 1525 6100 1525
+Wire Wire Line
+	7650 1525 7750 1525
+Wire Wire Line
+	6100 1825 6100 1775
+Wire Wire Line
+	6400 1825 6400 1775
+Wire Wire Line
+	6400 1575 6400 1525
+Wire Wire Line
+	6100 1575 6100 1525
+Connection ~ 6100 1525
+Wire Wire Line
+	6100 1525 6400 1525
+Wire Wire Line
+	6800 1825 6800 1775
+Wire Wire Line
+	6800 1575 6800 1525
+Wire Wire Line
+	7100 1825 7100 1775
+Wire Wire Line
+	7100 1575 7100 1525
+Connection ~ 7100 1525
+Wire Wire Line
+	7100 1525 7350 1525
+Wire Wire Line
+	7750 1575 7750 1525
+Connection ~ 7750 1525
+Wire Wire Line
+	7750 1525 8150 1525
+Wire Wire Line
+	7750 1825 7750 1775
+Wire Wire Line
+	8150 1825 8150 1775
+Wire Wire Line
+	8150 1575 8150 1525
+Wire Wire Line
+	7650 1525 7650 1975
 $EndSCHEMATC
