File: mark-II-Rpi-devkit/KiCAD/SJ201-Raspberry Pi 4 Daughterboard/xmos.sch (KiCad schematic (older format))
At the start: 59 parts, among them J10 Debug Connector, Q4 FDV301N, U10 MP34DT05, U11 MP34DT05, U12 NCP303LSN30, U5 74LVC125A, U7 AP3428A, U8 XMOS-XVF3510, U9 AT25SF161 16MBIT, X1 SG-210STF 24M

Commit message: Update BOM - fix OPL numbers for Seeed PCBA
Parts:
- PWR2: Link (none) -> https://lcsc.com/product-detail/Others_TOGIALED-TJ-S1608SW6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; MPN TJ-S1608SW6TGLC2R-A5 -> 19-217-R6C-AL1M2VY-3T; SKU (none) -> 304090042
Changed lines of the file:
@@
 F 2 "LED_SMD:LED_0603_1608Metric" H 3325 7075 50  0001 C CNN
 F 3 "https://datasheet.lcsc.com/szlcsc/1811141223_TOGIALED-TJ-S1608SW6TGLC2R-A5_C192315.pdf" H 3325 7075 50  0001 C CNN
-F 4 "TJ-S1608SW6TGLC2R-A5" H 3325 7075 50  0001 C CNN "MPN"
+F 4 "19-217-R6C-AL1M2VY-3T" H 3325 7075 50  0001 C CNN "MPN"
 F 5 "C192315" H 3325 7075 50  0001 C CNN "LCSC"
+F 6 "https://lcsc.com/product-detail/Others_TOGIALED-TJ-S1608SW6TGLC2R-A5_C192315.html" V 3325 7075 50  0001 C CNN "Link"
+F 7 "304090042" H 3325 7075 50  0001 C CNN "SKU"
 	1    3325 7075
 	-1   0    0    1

Commit message: Updated KiCAD files to 0.63 for PCB printing & Assembly at JLCPCB
Parts:
- removed C37, C39: 10UF, Capacitor_SMD:C_0402_1005Metric, symbol OPL_Capacitor:CERAMIC-2.2UF-25V-10%-X7R_0805_
- removed C38: 47pf, Capacitor_SMD:C_0402_1005Metric, symbol OPL_Capacitor:CERAMIC-2.2UF-25V-10%-X7R_0805_
- removed L3: 2.2UH-20%-1.2A_0805, OPL_Inductor:L0805, symbol OPL_Inductor:SMD-INDUCTOR-2.2UH-20%-1.2A_0805_
- removed R25: 47K, Resistor_SMD:R_0402_1005Metric, symbol Device:R_Small
- removed R37: 30K, Resistor_SMD:R_0402_1005Metric, symbol Device:R_Small
- removed U7: AP3428A, Package_TO_SOT_SMD:TSOT-23-5, symbol user:AP3428A
- added R5: 10R, Resistor_SMD:R_0402_1005Metric, symbol Device:R_Small
- C35, C36, C40, C41, C42, C43, C44, C45, C46, C47, C48, C49, C50, C51, C52, C53, C54, C57, C58: LCSC (none) -> C1525
- C55, C56: LCSC (none) -> C52923
- C65: LCSC (none) -> C1531
- C66: LCSC (none) -> C1523
- D20: LCSC (none) -> C179724-DNP
- FB5, FB6: footprint Resistor_SMD:R_0603_1608Metric -> Resistor_SMD:R_0805_2012Metric; LCSC (none) -> C1017
- PWR2: LCSC C192315 -> C2286
- Q4: LCSC (none) -> C15310
- R24: footprint Resistor_SMD:R_0402_1005Metric -> Resistor_SMD:R_0603_1608Metric; LCSC (none) -> C23164
- R26, R40: LCSC (none) -> C25792
- R32, R35, R36: LCSC (none) -> C25105
- R34: value 43R2 -> 33R; LCSC (none) -> C25105; MPN RC0402FR-0743R2L -> (none)
- R39, R52: LCSC (none) -> C25744
- R41: LCSC (none) -> C25900
- R43, R44, R45, R46: LCSC (none) -> C25076
- R53: LCSC (none) -> C25104
- U10, U11: value MP34DT05 -> SPK0838HT4H-1; Digikey 497-17809-1-ND -> 423-1432-1-ND; Link https://www.digikey.com/product-detail/en/stmicroelectronic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 -> https://www.digikey.com/product-detail/en/knowles/SPK0838HT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; MPN MP34DT05 -> SPK0838HT4H-1
- U12: LCSC (none) -> C146789
- U5: value 74LVC125A -> SN74LVC125APWR; footprint mycroft:DHVQFN14 -> Package_SO:TSSOP-14_4.4x5mm_P0.65mm; LCSC C282343 -> C7813; MPN 74LVC125ABQ,115 -> SN74LVC125APWR
- U9: LCSC (none) -> C93710
- X1: footprint Oscillator:Oscillator_SMD_SeikoEpson_SG210-4Pin_2.5x2.0mm -> Oscillator:Oscillator_SMD_SeikoEpson_SG8002CE-4Pin_3.2x2.5mm; LCSC (none) -> C32528
Connections:
- net labels removed: +5V
- wire segments 220 -> 204
Other:
- note added: "43R2 \ncombined \n2 Resistors"
- note added: "600R - LCSC"
- note removed: "VFB = 0.6V\nVO = 0.6 x (1 + 30/47) = 0.98V\n"

Commit message: Change USB IC to CM108B, add in Line Out jack, prep for 2 PCB sandwich
Parts:
- added J8: MIC, Connector_PinHeader_2.54mm:PinHeader_1x03_P2.54mm_Vertical, symbol Connector_Generic:Conn_01x03
Connections:
- net labels removed: I2S_BCK, I2S_DIN, MCLK
- wire segments 204 -> 192
Other:
- moved on the sheet: R39, R40, U5

Commit message: Mark 2 - PCB Files to the printer
Parts:
- U9: footprint Package_SO:SOIC-8_3.9x4.9mm_P1.27mm -> Package_SO:SOIC-8_5.23x5.23mm_P1.27mm
Changed lines of the file:
@@
 F 0 "U9" H 6950 2275 50  0000 C CNN
 F 1 "AT25SF161 16MBIT" H 7575 1775 50  0000 C CNN
-F 2 "Package_SO:SOIC-8_3.9x4.9mm_P1.27mm" H 7200 2025 50  0001 C CNN
+F 2 "Package_SO:SOIC-8_5.23x5.23mm_P1.27mm" H 7200 2025 50  0001 C CNN
 F 3 "http://ww1.microchip.com/downloads/en/DeviceDoc/Atmel-8707-SEEPROM-AT25010B-020B-040B-Datasheet.pdf" H 7200 2025 50  0001 C CNN
 F 4 "1265-1230-1-ND" H 7200 2025 50  0001 C CNN "Digikey"

Commit message: Update to v0.66 - printed at JLC - 2nd spin
Parts:
- removed TP1_0V1: TestPoint, TestPoint:TestPoint_Pad_D1.0mm, symbol Connector:TestPoint
- added R9: 4.7k, Resistor_SMD:R_0402_1005Metric, symbol Device:R_Small
- added TP28: TestPoint, TestPoint:TestPoint_Pad_D2.0mm, symbol Connector:TestPoint
- U12: value NCP303LSN30 -> NCP303LSN09; LCSC C146789 -> C150075; MPN NCP303LSN30T1G -> NCP303LSN09T1G
- U8: footprint user:QFN-60-1EP_7x7mm_P0.4mm_EP5.6x5.6mm -> user:QFN-60-1EP_7x7mm_P0.4mm_EP5.6x5.6mm-HandSolder
Connections:
- wire segments 192 -> 193
- no-connect marks 10 -> 9
Other:
- moved on the sheet: X1
Changed lines of the file:
@@
 Sheet 6 6
 Title ""
-Date "2020-07-24"
-Rev "0.65"
+Date "2020-08-16"
+Rev "0.66"
 Comp ""
 Comment1 ""
@@
 L Oscillator:SG-210STF X1
 U 1 1 5F20B513
-P 850 3250
-F 0 "X1" H 950 3500 50  0000 L CNN
-F 1 "SG-210STF 24M" H 925 3000 50  0000 L CNN
-F 2 "Oscillator:Oscillator_SMD_SeikoEpson_SG8002CE-4Pin_3.2x2.5mm" H 1300 2900 50  0001 C CNN
-F 3 "https://support.epson.biz/td/api/doc_check.php?mode=dl&lang=en&Parts=SG-210STF" H 750 3250 50  0001 C CNN
-F 4 "SG-210STF 24M" H 850 3250 50  0001 C CNN "MPN"
-F 5 "https://www.digikey.com/product-detail/en/epson/SG-210STF-24.0000ML3/SER4323CT-ND/7932310" H 850 3250 50  0001 C CNN "Link"
-F 6 "C32528" H 850 3250 50  0001 C CNN "LCSC"
-	1    850  3250
+P 975 3250
+F 0 "X1" H 1075 3500 50  0000 L CNN
+F 1 "SG-210STF 24M" H 1050 3000 50  0000 L CNN
+F 2 "Oscillator:Oscillator_SMD_SeikoEpson_SG8002CE-4Pin_3.2x2.5mm" H 1425 2900 50  0001 C CNN
+F 3 "https://support.epson.biz/td/api/doc_check.php?mode=dl&lang=en&Parts=SG-210STF" H 875 3250 50  0001 C CNN
+F 4 "SG-210STF 24M" H 975 3250 50  0001 C CNN "MPN"
+F 5 "https://www.digikey.com/product-detail/en/epson/SG-210STF-24.0000ML3/SER4323CT-ND/7932310" H 975 3250 50  0001 C CNN "Link"
+F 6 "C32528" H 975 3250 50  0001 C CNN "LCSC"
+	1    975  3250
 	1    0    0    -1
 $EndComp
@@
 L power:GND #PWR?
 U 1 1 5F20CBD6
-P 850 3550
+P 975 3550
 AR Path="/5EA9C461/5F20CBD6" Ref="#PWR?"  Part="1"
 AR Path="/5EA9C67D/5F20CBD6" Ref="#PWR?"  Part="1"
 AR Path="/5EA9C76D/5F20CBD6" Ref="#PWR066"  Part="1"
-F 0 "#PWR066" H 850 3300 50  0001 C CNN
-F 1 "GND" H 855 3377 50  0000 C CNN
-F 2 "" H 850 3550 50  0001 C CNN
-F 3 "" H 850 3550 50  0001 C CNN
-	1    850  3550
+F 0 "#PWR066" H 975 3300 50  0001 C CNN
+F 1 "GND" H 980 3377 50  0000 C CNN
+F 2 "" H 975 3550 50  0001 C CNN
+F 3 "" H 975 3550 50  0001 C CNN
+	1    975  3550
 	1    0    0    -1
 $EndComp
-Wire Wire Line
-	1450 3250 1150 3250
-NoConn ~ 550  3250
 $Comp
 L power:+3.3V #PWR065
 U 1 1 5F20F77E
-P 850 2950
-F 0 "#PWR065" H 850 2800 50  0001 C CNN
-F 1 "+3.3V" H 865 3123 50  0000 C CNN
-F 2 "" H 850 2950 50  0001 C CNN
-F 3 "" H 850 2950 50  0001 C CNN
-	1    850  2950
+P 975 2950
+F 0 "#PWR065" H 975 2800 50  0001 C CNN
+F 1 "+3.3V" H 990 3123 50  0000 C CNN
+F 2 "" H 975 2950 50  0001 C CNN
+F 3 "" H 975 2950 50  0001 C CNN
+	1    975  2950
 	1    0    0    -1
 $EndComp
@@
 	4025 2950 4725 2950
 Wire Wire Line
-	4725 3150 4025 3150
-Wire Wire Line
 	4025 3250 4725 3250
 Wire Wire Line
@@
 F 0 "U8" H 2700 1400 55  0000 L CNN
 F 1 "XMOS-XVF3510" H 2700 -2750 55  0000 L CNN
-F 2 "user:QFN-60-1EP_7x7mm_P0.4mm_EP5.6x5.6mm" H 3275 1350 55  0001 C CNN
+F 2 "user:QFN-60-1EP_7x7mm_P0.4mm_EP5.6x5.6mm-HandSolder" H 3275 1350 55  0001 C CNN
 F 3 "" H 3275 1350 55  0001 C CNN
 F 4 "XVF3510" H 3275 1350 50  0001 C CNN "MPN"
@@
 Wire Wire Line
 	4725 2850 4025 2850
-Wire Wire Line
-	4025 3050 4725 3050
 Text Label 8975 1825 0    51   ~ 0
 3V3_MIC
@@
 Power on RESET
 $Comp
-L user:NCP303LSN30 U12
-U 1 1 5F0AC355
-P 1825 7300
-F 0 "U12" H 1900 7668 51  0000 C CNN
-F 1 "NCP303LSN30" H 1900 7575 51  0000 C CNN
-F 2 "Package_TO_SOT_SMD:SOT-23-5" H 1825 7300 51  0001 C CNN
-F 3 "https://www.onsemi.com/pub/Collateral/NCP302-D.PDF" H 1825 7300 51  0001 C CNN
-F 4 "NCP303LSN30T1G" H 1825 7300 50  0001 C CNN "MPN"
-F 5 "C146789" H 1825 7300 50  0001 C CNN "LCSC"
-	1    1825 7300
-	1    0    0    -1
-$EndComp
-$Comp
 L power:GND #PWR?
 U 1 1 5F0ACBA1
@@
 $EndComp
 $Comp
-L power:+3.3V #PWR030
-U 1 1 5F0ACF0B
-P 1375 7200
-F 0 "#PWR030" H 1375 7050 50  0001 C CNN
-F 1 "+3.3V" H 1390 7373 50  0000 C CNN
-F 2 "" H 1375 7200 50  0001 C CNN
-F 3 "" H 1375 7200 50  0001 C CNN
-	1    1375 7200
-	1    0    0    -1
-$EndComp
-$Comp
 L OPL_Capacitor:CERAMIC-2.2UF-25V-10%-X7R_0805_ C?
 U 1 1 5F0B0062
@@
 Wire Notes Line
 	600  6700 600  7775
-$Comp
-L Connector:TestPoint TP?
-U 1 1 5F15149B
-P 700 5325
-AR Path="/5EA9C461/5F15149B" Ref="TP?"  Part="1"
-AR Path="/5EA9C76D/5F15149B" Ref="TP1_0V1"  Part="1"
-F 0 "TP1_0V1" V 775 5600 50  0000 R CNN
-F 1 "TestPoint" V 700 6075 50  0001 R CNN
-F 2 "TestPoint:TestPoint_Pad_D1.0mm" H 900 5325 50  0001 C CNN
-F 3 "~" H 900 5325 50  0001 C CNN
-	1    700  5325
-	0    1    1    0
-$EndComp
-$Comp
-L power:+1V0 #PWR038
-U 1 1 5F1614D7
-P 700 5325
-F 0 "#PWR038" H 700 5175 50  0001 C CNN
-F 1 "+1V0" H 715 5498 50  0000 C CNN
-F 2 "" H 700 5325 50  0001 C CNN
-F 3 "" H 700 5325 50  0001 C CNN
-	1    700  5325
-	1    0    0    -1
-$EndComp
 Text Notes 9275 2075 0    50   ~ 0
 600R - LCSC
@@
 Wire Wire Line
 	4175 1450 4025 1450
+$Comp
+L power:+1V0 #PWR0163
+U 1 1 5F3A4147
+P 1375 7200
+F 0 "#PWR0163" H 1375 7050 50  0001 C CNN
+F 1 "+1V0" H 1390 7373 50  0000 C CNN
+F 2 "" H 1375 7200 50  0001 C CNN
+F 3 "" H 1375 7200 50  0001 C CNN
+	1    1375 7200
+	1    0    0    -1
+$EndComp
+$Comp
+L user:NCP303LSN30 U12
+U 1 1 5F0AC355
+P 1825 7300
+F 0 "U12" H 1900 7668 51  0000 C CNN
+F 1 "NCP303LSN09" H 1900 7575 51  0000 C CNN
+F 2 "Package_TO_SOT_SMD:SOT-23-5" H 1825 7300 51  0001 C CNN
+F 3 "https://www.onsemi.com/pub/Collateral/NCP302-D.PDF" H 1825 7300 51  0001 C CNN
+F 4 "NCP303LSN09T1G" H 1825 7300 50  0001 C CNN "MPN"
+F 5 "C150075" H 1825 7300 50  0001 C CNN "LCSC"
+	1    1825 7300
+	1    0    0    -1
+$EndComp
+$Comp
+L power:+3.3V #PWR0164
+U 1 1 5F3F8955
+P 600 3250
+F 0 "#PWR0164" H 600 3100 50  0001 C CNN
+F 1 "+3.3V" H 615 3423 50  0000 C CNN
+F 2 "" H 600 3250 50  0001 C CNN
+F 3 "" H 600 3250 50  0001 C CNN
+	1    600  3250
+	1    0    0    -1
+$EndComp
+Wire Wire Line
+	675  3250 600  3250
+Wire Wire Line
+	1275 3250 1450 3250
+$Comp
+L Device:R_Small R?
+U 1 1 5F417201
+P 4950 2950
+AR Path="/5EA9C461/5F417201" Ref="R?"  Part="1"
+AR Path="/5EA9C67D/5F417201" Ref="R?"  Part="1"
+AR Path="/5EA9C76D/5F417201" Ref="R9"  Part="1"
+F 0 "R9" V 5025 2875 50  0000 L CNN
+F 1 "4.7k" V 4875 2850 50  0000 L CNN
+F 2 "Resistor_SMD:R_0402_1005Metric" H 4950 2950 50  0001 C CNN
+F 3 "~" H 4950 2950 50  0001 C CNN
+F 4 "0402WGF4701TCE" H 4950 2950 50  0001 C CNN "MPN"
+F 5 "C25900" H 4950 2950 50  0001 C CNN "LCSC"
+	1    4950 2950
+	-1   0    0    1
+$EndComp
+$Comp
+L Connector:TestPoint TP28
+U 1 1 5F417FE4
+P 4950 2850
+F 0 "TP28" H 5008 2968 50  0000 L CNN
+F 1 "TestPoint" H 5008 2877 50  0000 L CNN
+F 2 "TestPoint:TestPoint_Pad_D2.0mm" H 5150 2850 50  0001 C CNN
+F 3 "~" H 5150 2850 50  0001 C CNN
+	1    4950 2850
+	1    0    0    -1
+$EndComp
+Wire Wire Line
+	4725 3150 4025 3150
+Wire Wire Line
+	4025 3050 4950 3050
 $EndSCHEMATC

Commit message: Fix missing items in schematic in Github
Parts:
- C35, C36, C40, C41, C42, C43, C44, C45, C46, C47, C48, C49, C50, C51, C52, C53, C54, C55, C56, C57, C58: symbol OPL_Capacitor:CERAMIC-100NF-50V-10%-X7R_0805_ -> Device:C_Small
- C65, C66: symbol OPL_Capacitor:CERAMIC-2.2UF-25V-10%-X7R_0805_ -> Device:C_Small
Connections:
- wire segments 193 -> 237
