File: mark-II-Rpi-devkit/KiCAD/SJ201-Raspberry Pi 4 Daughterboard/xmos.sch (KiCad schematic (older format))
At the start: 63 parts, among them U10 SPK0641HT4H-1, U11 SPK0641HT4H-1, U5 SN74LVC125APWR, U8 XMOS-XVF3510, U9 DNP - AT25SFxx 16mb or greater, X1 SG-210STF 24M

Commit message: Removed unused files, cleaned up directory, remove SJ202
Parts:
- FB5, FB6: symbol kevin:Ferrite_Bead_Small -> Mycroft:Ferrite_Bead_Small
- U10, U11: footprint user:HCLGA-MP34DT05 -> Mycroft:HCLGA-MP34DT05
- U5: symbol user:74LVC125A -> Mycroft:74LVC125A
- U8: footprint user:QFN-60-1EP_7x7mm_P0.4mm_EP5.6x5.6mm -> XMOS:QFN-60-1EP_7x7mm_P0.4mm_EP5.6x5.6mm; symbol user:XMOS-XVF3510 -> Mycroft:XMOS-XVF3510
Changed lines of the file:
@@
 $EndComp
 $Comp
-L kevin:Ferrite_Bead_Small FB5
+L Mycroft:Ferrite_Bead_Small FB5
 U 1 1 5F43B8E2
 P 8850 1825
@@
 Alternate Mic part #:\nSPK0838HT4H-1
 $Comp
-L kevin:Ferrite_Bead_Small FB6
+L Mycroft:Ferrite_Bead_Small FB6
 U 1 1 5F22AB88
 P 8850 2650
@@
 F 0 "U10" H 8372 3521 50  0000 R CNN
 F 1 "SPK0641HT4H-1" H 8550 2975 50  0000 R CNN
-F 2 "user:HCLGA-MP34DT05" H 8150 3800 50  0001 L BNN
+F 2 "Mycroft:HCLGA-MP34DT05" H 8150 3800 50  0001 L BNN
 F 3 "https://www.knowles.com/docs/default-source/model-downloads/spk0641ht4h-1-rev-a.pdf" H 8650 3550 63  0001 C CNN
 F 4 "423-1425-1-ND" H 8700 3600 50  0001 C CNN "Digikey"
@@
 F 0 "U11" H 8372 4846 50  0000 R CNN
 F 1 "SPK0641HT4H-1" H 8600 4300 50  0000 R CNN
-F 2 "user:HCLGA-MP34DT05" H 8150 5125 50  0001 L BNN
+F 2 "Mycroft:HCLGA-MP34DT05" H 8150 5125 50  0001 L BNN
 F 3 "https://www.knowles.com/docs/default-source/model-downloads/spk0641ht4h-1-rev-a.pdf" H 8650 4875 63  0001 C CNN
 F 4 "423-1425-1-ND" H 8700 4925 50  0001 C CNN "Digikey"
@@
 	2475 4350 2325 4350
 $Comp
-L user:XMOS-XVF3510 U8
+L Mycroft:XMOS-XVF3510 U8
 U 1 1 5F1E8ACB
 P 3275 1350
 F 0 "U8" H 2700 1400 55  0000 L CNN
 F 1 "XMOS-XVF3510" H 2700 -2750 55  0000 L CNN
-F 2 "user:QFN-60-1EP_7x7mm_P0.4mm_EP5.6x5.6mm" H 3275 1350 55  0001 C CNN
+F 2 "XMOS:QFN-60-1EP_7x7mm_P0.4mm_EP5.6x5.6mm" H 3275 1350 55  0001 C CNN
 F 3 "" H 3275 1350 55  0001 C CNN
 F 4 "XVF3510-QF60-C" H 3275 1350 50  0001 C CNN "MPN"
@@
 $EndComp
 $Comp
-L user:74LVC125A U5
+L Mycroft:74LVC125A U5
 U 1 1 5F0C90C8
 P 6325 4800
