File: mark-II-Rpi-devkit/KiCAD/SJ201-Raspberry Pi 4 Daughterboard/AudioAmp.sch (KiCad schematic (older format))
At the start: 56 parts, among them J2 PVDD Jumper, J3 SPKLEFT, J4 SPKRIGHT, U2 PCM2706, U3 MAX9744, Y1 12MHz

Commit message: Update BOM - fix OPL numbers for Seeed PCBA
Parts:
- C13, C14, C24, C25, C26, C27: SKU (none) -> 508000001
Changed lines of the file:
@@
 F 3 "http://file.elecfans.com/web1/M00/7D/4D/o4YBAFwKKSOANZPCAA-X9Qix-h8480.pdf" H 3650 2000 50  0001 C CNN
 F 4 "0402B471K500NT" H 3680 2150 20  0001 C CNN "MPN"
+F 5 "508000001" H 3650 2000 50  0001 C CNN "SKU"
 	1    3650 2000
 	1    0    0    -1
@@
 F 3 "http://file.elecfans.com/web1/M00/7D/4D/o4YBAFwKKSOANZPCAA-X9Qix-h8480.pdf" H 3650 2400 50  0001 C CNN
 F 4 "0402B471K500NT" H 3680 2550 20  0001 C CNN "MPN"
+F 5 "508000001" H 3650 2400 50  0001 C CNN "SKU"
 	1    3650 2400
 	1    0    0    -1
@@
 F 3 "http://file.elecfans.com/web1/M00/7D/4D/o4YBAFwKKSOANZPCAA-X9Qix-h8480.pdf" H 8200 2250 50  0001 C CNN
 F 4 "0402B471K500NT" H 8230 2400 20  0001 C CNN "MPN"
-F 5 "" H 8230 2400 20  0001 C CNN "SKU"
+F 5 "508000001" H 8230 2400 20  0001 C CNN "SKU"
 	1    8200 2250
 	1    0    0    -1
@@
 F 3 "http://file.elecfans.com/web1/M00/7D/4D/o4YBAFwKKSOANZPCAA-X9Qix-h8480.pdf" H 7800 2250 50  0001 C CNN
 F 4 "0402B471K500NT" H 7830 2400 20  0001 C CNN "MPN"
-F 5 "" H 7830 2400 20  0001 C CNN "SKU"
+F 5 "508000001" H 7830 2400 20  0001 C CNN "SKU"
 	1    7800 2250
 	1    0    0    -1
@@
 F 3 "http://file.elecfans.com/web1/M00/7D/4D/o4YBAFwKKSOANZPCAA-X9Qix-h8480.pdf" H 7800 2950 50  0001 C CNN
 F 4 "0402B471K500NT" H 7830 3100 20  0001 C CNN "MPN"
-F 5 "" H 7830 3100 20  0001 C CNN "SKU"
+F 5 "508000001" H 7830 3100 20  0001 C CNN "SKU"
 	1    7800 2950
 	1    0    0    -1
@@
 F 3 "http://file.elecfans.com/web1/M00/7D/4D/o4YBAFwKKSOANZPCAA-X9Qix-h8480.pdf" H 8200 2950 50  0001 C CNN
 F 4 "0402B471K500NT" H 8230 3100 20  0001 C CNN "MPN"
-F 5 "" H 8230 3100 20  0001 C CNN "SKU"
+F 5 "508000001" H 8230 3100 20  0001 C CNN "SKU"
 	1    8200 2950
 	1    0    0    -1

Commit message: Updated KiCAD files to 0.63 for PCB printing & Assembly at JLCPCB
Parts:
- added U13: CM108AH, QFP50P900X900X160-48N, symbol CM108AH:CM108AH
- added U14: TAS5711PHPR, Texas_Instruments-TAS5711PHPR-*, symbol eec:TAS5711PHPR
- C10: footprint OPL_Capacitor:AVX-A(1206) -> Capacitor_Tantalum_SMD:CP_EIA-3216-18_Kemet-A; symbol OPL_Capacitor:TANTALUM-SMD-10UF-10V-10%_AVX-A_ -> Device:CP; LCSC (none) -> C7171
- C11, C12, C15, C16, C61, C9: LCSC (none) -> C52923
- C13, C14, C24, C25, C26, C27: LCSC (none) -> C1537
- C17, C18, C19, C20, C21, C22: LCSC (none) -> C1525
- C23: footprint Capacitor_SMD:C_0402_1005Metric -> Capacitor_SMD:C_0603_1608Metric; LCSC (none) -> C23630
- C62: footprint user:CP_Elec_8x10.5_OPL -> Capacitor_SMD:CP_Elec_8x10.5; symbol OPL_Capacitor:DIP-ALUMINUM-47UF-16V_D5-H7MM_ -> Device:CP; LCSC (none) -> C176671
- FB1, FB2, FB3, FB4, FB7: footprint Resistor_SMD:R_0805_2012Metric -> Resistor_SMD:R_1206_3216Metric; LCSC (none) -> C29107; MPN MPZ2012S101AT000 -> MLB3216-301P3A(f)
- R10: LCSC (none) -> C26083
- R11, R19: LCSC (none) -> C25867
- R12, R13, R14, R15, R16, R9: LCSC (none) -> C25092
- R17, R18, R21, R22: LCSC (none) -> C25765
- R20, R42, R47, R48, R49, R50, R51: LCSC (none) -> C25744
Connections:
- net labels added: I2S_BCLK, I2S_DIN, I2S_DOUT, MCLK
- wire segments 205 -> 222
Other:
- note added: "CM108AH- change part"
- note added: "Change part to \nTAS5711PHPR"
- note added: "I2S Data from \nUSB Soundcard"

Commit message: Change USB IC to CM108B, add in Line Out jack, prep for 2 PCB sandwich
Parts:
- removed C10: 10UF, Capacitor_Tantalum_SMD:CP_EIA-3216-18_Kemet-A, symbol Device:CP
- removed C11, C12, C15, C16, C9: 1uF, Capacitor_SMD:C_0402_1005Metric, symbol OPL_Capacitor:CERAMIC-100NF-50V-10%-X7R_0805_
- removed R10: 1M, Resistor_SMD:R_0402_1005Metric, symbol Device:R_Small
- removed R11, R19: 1k5, Resistor_SMD:R_0402_1005Metric, symbol Device:R_Small
- removed R12, R13, R14, R15, R16, R9: 22R, Resistor_SMD:R_0402_1005Metric, symbol Device:R_Small
- removed U14: TAS5711PHPR, Texas_Instruments-TAS5711PHPR-*, symbol eec:TAS5711PHPR
- removed U2: PCM2706, Package_QFP:TQFP-32_7x7mm_P0.8mm, symbol user:PCM2706
- removed Y1: 12MHz, Crystal:Crystal_SMD_3225-4Pin_3.2x2.5mm, symbol Device:Crystal_GND23
- added C38: 4.7UF, Capacitor_SMD:C_0402_1005Metric, symbol OPL_Capacitor:CERAMIC-2.2UF-25V-10%-X7R_0805_
- added J11: I2S, Connector_PinHeader_2.54mm:PinHeader_1x04_P2.54mm_Vertical, symbol Connector_Generic:Conn_01x04
- added J9: AudioJack3_Ground_Switch, mycroft:STX-3790-5N, symbol Connector:AudioJack2_Ground_Switch
- added R25, R37: 22R, Resistor_SMD:R_0402_1005Metric, symbol Device:R_Small
- added R6: 330R, Resistor_SMD:R_0402_1005Metric, symbol Device:R_Small
- added R7: 1k5, Resistor_SMD:R_0402_1005Metric, symbol Device:R_Small
- added USB_GP1, USB_GP3, USB_GP4: TestPoint, TestPoint:TestPoint_Pad_D1.0mm, symbol Connector:TestPoint
- added USB_SOUND1: LED, LED_SMD:LED_0603_1608Metric, symbol Device:LED
- C62: LCSC C176671 -> C176671-DNP
- U13: value CM108AH -> CM108B; footprint QFP50P900X900X160-48N -> Package_QFP:LQFP-48_7x7mm_P0.5mm; symbol CM108AH:CM108AH -> CM108AH:CM108B; LCSC (none) -> C371347
Connections:
- net labels added: AREG36, DREG33
- net labels removed: HID0, HID1, HID2, VDD
- wire segments 222 -> 166
- no-connect marks 3 -> 22
Other:
- note added: "EEPROM"
- note added: "Ignore all ADC \nclock and inputs"
- note added: "MSEL ignored"
- note removed: "CM108AH- change part"
- moved on the sheet: C13, C14, R51, TP22, TP23

Commit message: Update to v0.66 - printed at JLC - 2nd spin
Parts:
- TP22, TP23, TP24: footprint TestPoint:TestPoint_Pad_D1.0mm -> TestPoint:TestPoint_Pad_D2.0mm
Changed lines of the file:
@@
 Sheet 3 6
 Title ""
-Date "2020-07-24"
-Rev "0.65"
+Date "2020-08-16"
+Rev "0.66"
 Comp "Mycroft"
 Comment1 ""
@@
 F 0 "TP24" V 3200 3150 50  0000 R CNN
 F 1 "TestPoint" V 3200 3550 50  0001 R CNN
-F 2 "TestPoint:TestPoint_Pad_D1.0mm" H 3400 2800 50  0001 C CNN
+F 2 "TestPoint:TestPoint_Pad_D2.0mm" H 3400 2800 50  0001 C CNN
 F 3 "~" H 3400 2800 50  0001 C CNN
 	1    3200 2800
@@
 F 0 "TP23" H 3725 2625 50  0000 R CNN
 F 1 "TestPoint" V 3675 3150 50  0001 R CNN
-F 2 "TestPoint:TestPoint_Pad_D1.0mm" H 3875 2400 50  0001 C CNN
+F 2 "TestPoint:TestPoint_Pad_D2.0mm" H 3875 2400 50  0001 C CNN
 F 3 "~" H 3875 2400 50  0001 C CNN
 	1    3675 2400
@@
 F 0 "TP22" H 3750 2200 50  0000 R CNN
 F 1 "TestPoint" V 3675 2750 50  0001 R CNN
-F 2 "TestPoint:TestPoint_Pad_D1.0mm" H 3875 2000 50  0001 C CNN
+F 2 "TestPoint:TestPoint_Pad_D2.0mm" H 3875 2000 50  0001 C CNN
 F 3 "~" H 3875 2000 50  0001 C CNN
 	1    3675 2000

Commit message: Fix missing items in schematic in Github
Parts:
- C13, C14, C17, C18, C19, C20, C21, C22, C24, C25, C26, C27, C61: symbol OPL_Capacitor:CERAMIC-100NF-50V-10%-X7R_0805_ -> Device:C_Small
- C23, C38: symbol OPL_Capacitor:CERAMIC-2.2UF-25V-10%-X7R_0805_ -> Device:C_Small
Connections:
- wire segments 166 -> 176

Commit message: SJ201 - Removed CM108b soundcard, added in I2S to Line out, ATTin402. Moved holes in layout. SJ202 - extened length to plug into USB2.0 port
Parts:
- removed C13: 470pF, Capacitor_SMD:C_0402_1005Metric, symbol Device:C_Small
- removed C38: 4.7UF, Capacitor_SMD:C_0402_1005Metric, symbol Device:C_Small
- removed R25, R37: 22R, Resistor_SMD:R_0402_1005Metric, symbol Device:R_Small
- removed TP24: TestPoint, TestPoint:TestPoint_Pad_D2.0mm, symbol Connector:TestPoint
- removed U13: CM108B, Package_QFP:LQFP-48_7x7mm_P0.5mm, symbol CM108AH:CM108B
- removed USB_GP1, USB_GP3, USB_GP4: TestPoint, TestPoint:TestPoint_Pad_D1.0mm, symbol Connector:TestPoint
- removed USB_SOUND1: LED, LED_SMD:LED_0603_1608Metric, symbol Device:LED
- added C10: 100NF, Capacitor_SMD:C_0402_1005Metric, symbol Device:C_Small
- added C11: 10UF, Capacitor_SMD:C_0402_1005Metric, symbol Device:C_Small
- added C12, C13: 47UF/16V, Capacitor_SMD:CP_Elec_5x5.3, symbol Device:CP
- added C15: 10nF, Capacitor_SMD:C_0402_1005Metric, symbol Device:C_Small
- added C16: 22pFDNP, Capacitor_SMD:C_0402_1005Metric, symbol Device:C_Small
- added FB9: FB, Resistor_SMD:R_1206_3216Metric, symbol kevin:Ferrite_Bead_Small
- added J12: SCL, Jumper:SolderJumper-3_P1.3mm_Bridged2Bar12_RoundedPad1.0x1.5mm_NumberLabels, symbol Connector_Generic:Conn_01x03
- added J14: SDA, Jumper:SolderJumper-3_P1.3mm_Bridged2Bar12_RoundedPad1.0x1.5mm_NumberLabels, symbol Connector_Generic:Conn_01x03
- added R10, R11: 100R, Resistor_SMD:R_0402_1005Metric, symbol Device:R_Small
- added U13: UDA1334ATS, Package_SO:SSOP-16_4.4x5.2mm_P0.65mm, symbol Audio:UDA1334ATS
- C14: value 470pF -> 10nF; LCSC C1537 -> C15195; MPN 0402B471K500NT -> CL05B103KB5NNNC; SKU 508000001 -> (none)
- C61: MPN CC0402KRX5R6BB105 -> CL05A105KA5NQNC; SKU 302010040 -> (none)
- J11: footprint Connector_PinHeader_2.54mm:PinHeader_1x04_P2.54mm_Vertical -> Connector_PinHeader_2.54mm:PinHeader_1x05_P2.54mm_Vertical; symbol Connector_Generic:Conn_01x04 -> Connector_Generic:Conn_01x05; MPN (none) -> DNP
- J2, NT1, TP22, TP23: MPN (none) -> DNP
- J3: Link (none) -> https://www.newark.com/jst-japan-solderless-terminals/b2b-p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; MPN (none) -> B2B-PH-SM4-TB(LF)(SN); Vendor (none) -> Newark
- J4: Link (none) -> https://www.newark.com/jst-japan-solderless-terminals/b2b-p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; MPN (none) -> B2B-PH-SM4-TB(LF)(SN)
- J9: Digikey (none) -> 2092-STX-3790-5N-ND; Link (none) -> https://www.digikey.com/product-detail/en/kycon-inc/STX-379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; MPN (none) -> DNP
- R6: value 330R -> 220k; LCSC C25104 -> C25767; MPN 0402WGF3300TCE -> 0402WGF2203TCE
- R7: value 1k5 -> 220k; LCSC C25867 -> C25767; MPN 0402WGF1501TCE -> 0402WGF2203TCE
Connections:
- net labels added: SCL, SCL_XMOS, SDA, SDA_XMOS
- net labels removed: +5V, AREG36, DREG33, GNDA, USB_SOUNDCARD_D+, USB_SOUNDCARD_D-
- wire segments 176 -> 212
- no-connect marks 22 -> 0
Other:
- note added: "Default to RasPi I2C.\nCut jumper between 1 & 2 \nand solder 2 to 3\nto enable XMOS I2C"
- note added: "I2S to Line Out"
- note added: "https://learn.adafruit.com/assets/48419"
- note removed: "EEPROM"
- note removed: "Ignore all ADC \nclock and inputs"
- note removed: "MSEL ignored"
- note removed: "http://www.pavouk.org/hw/audiosystem20/en_pcm2706usbi2s.html\n\nhttp://www.pavouk.org/hw/audiosystem20/pcm2706_usb_i2s_sch.pdf"
