File: mark-II-Rpi-devkit/KiCAD/SJ201-Raspberry Pi 4 Daughterboard/AudioAmp.sch (KiCad schematic (older format))
At the start: 53 parts, among them J11 I2S, J12 SCL, J14 SDA, J2 PVDD Jumper, J3 SPKLEFT, J4 SPKRIGHT, J9 AudioJack3_Ground_Switch, U13 UDA1334ATS, U3 MAX9744

Commit message: SJ-201 v3, sent to PCB Fab. Removed USB Hub, add in I2S to Line Out
Parts:
- removed J12: SCL, Jumper:SolderJumper-3_P1.3mm_Bridged2Bar12_RoundedPad1.0x1.5mm_NumberLabels, symbol Connector_Generic:Conn_01x03
- removed J14: SDA, Jumper:SolderJumper-3_P1.3mm_Bridged2Bar12_RoundedPad1.0x1.5mm_NumberLabels, symbol Connector_Generic:Conn_01x03
- removed J2: PVDD Jumper, Jumper:SolderJumper-2_P1.3mm_Bridged_RoundedPad1.0x1.5mm, symbol Connector_Generic:Conn_01x02
- added R25, R37: 0R - DNP, Resistor_SMD:R_0603_1608Metric, symbol Device:R_Small
- added R54, R55: 0R, Resistor_SMD:R_0603_1608Metric, symbol Device:R_Small
- added R56: 0R, Resistor_SMD:R_1206_3216Metric, symbol Device:R_Small
- C12, C13: LCSC C134798 -> C134798-DNP; Tempo (none) -> RVS-6V470MU-R
- C23: MPN CC0402MRX5R5BB225 -> EMK107BJ225KA-T
- C24, C25, C26, C27: SKU 508000001 -> (none); Tempo (none) -> GRM155R71H471KA01D
- C62: Tempo (none) -> EEE-1CA471UP
- FB1, FB2, FB3, FB4, FB7, FB9: Tempo (none) -> BK32164S301-T
- J3: value SPKLEFT -> SPK
- J4: value SPKRIGHT -> SPK
- R10, R11: Tempo (none) -> RC0402FR-07100RL
- R17, R18, R21, R22: Tempo (none) -> RC0402FR-0720KL
- R6, R7: Tempo (none) -> ERJ-2GEJ224X
Connections:
- net labels added: GNDA
- wire segments 212 -> 221
Other:
- note added: "I2C Selector"
- note added: "I2C Selector\nPopulate:\nR54 and R55 for Raspi\nR25 and R37 for XMOS"
- note added: "Left"
- note added: "PVDD Jumper"
- note added: "Right"
- note removed: "Default to RasPi I2C.\nCut jumper between 1 & 2 \nand solder 2 to 3\nto enable XMOS I2C"

Commit message: Rev4 Update - Add in Coral TPU, TAS5806, remove I2S * MAX9744. Change Attiny to Attin1614
Parts:
- removed C12, C13: 47UF/16V, Capacitor_SMD:CP_Elec_5x5.3, symbol Device:CP
- removed C62: 470UF/16V, Capacitor_SMD:CP_Elec_8x10.5, symbol Device:CP
- removed FB7, FB9: FB, Resistor_SMD:R_1206_3216Metric, symbol kevin:Ferrite_Bead_Small
- removed J11: I2S, Connector_PinHeader_2.54mm:PinHeader_1x05_P2.54mm_Vertical, symbol Connector_Generic:Conn_01x05
- removed NT1: Net-Tie_2, NetTie:NetTie-2_SMD_Pad0.5mm, symbol Device:Net-Tie_2
- removed R10, R11: 100R, Resistor_SMD:R_0402_1005Metric, symbol Device:R_Small
- removed R17, R18, R21, R22: 20k, Resistor_SMD:R_0402_1005Metric, symbol Device:R_Small
- removed R20, R42, R51: 10k, Resistor_SMD:R_0402_1005Metric, symbol Device:R_Small
- removed TP22, TP23: TestPoint, TestPoint:TestPoint_Pad_D2.0mm, symbol Connector:TestPoint
- removed U13: UDA1334ATS, Package_SO:SSOP-16_4.4x5.2mm_P0.65mm, symbol Audio:UDA1334ATS
- removed U3: MAX9744, max9744:max9744eth&plus_, symbol user:MAX9744ETH_T
- added C12: 100NF, Capacitor_SMD:C_0402_1005Metric, symbol Device:C_Small
- added C13: 22UF, Capacitor_SMD:C_0603_1608Metric, symbol Device:C_Small
- added C38, C39, C62: 1NF, Capacitor_SMD:C_0402_1005Metric, symbol Device:C_Small
- added R16, R53, R62: 0R, Resistor_SMD:R_0402_1005Metric, symbol Device:R_Small
- added R52, R63: 0R - DNP, Resistor_SMD:R_0402_1005Metric, symbol Device:R_Small
- added R64, R65, R66: 33R, Resistor_SMD:R_0402_1005Metric, symbol Device:R_Small
- added TP1, TP3, TP4: TestPoint, TestPoint:TestPoint_Pad_D1.0mm, symbol Connector:TestPoint
- added U14: NC7NZ34K8XTR, NC7N:ON_Semi-NZ34-0-0-0, symbol nc7nz:NC7NZ34K8X
- added U3: TAS5806MD, TAS5806MD:TAS5806MDDCPR, symbol TAS5806MD:TAS5806MDDCPR
- C10: value 100NF -> 4.7UF; LCSC C1525 -> C23733; MPN CC0402KRX7R8BB104 -> CL05A475MP5NRNC; SKU 302010024 -> (none)
- C11: value 10UF -> 100NF; LCSC C15525 -> C1525; MPN CC0402MRX5R5BB106 -> CC0402KRX7R8BB104; SKU 302010053 -> 302010024
- C14: value 10nF -> 22UF; footprint Capacitor_SMD:C_0402_1005Metric -> Capacitor_SMD:C_0603_1608Metric; LCSC C15195 -> C59461; MPN CL05B103KB5NNNC -> CL10A226MQ8NRNC
- C15: value 10nF -> 1uF; LCSC C15195 -> C52923; MPN CL05B103KB5NNNC -> CL05A105KA5NQNC
- C16: value 22pFDNP -> 1uF; LCSC DNP C1555 -> C52923; MPN DNP - 0402CG220J500NT -> CL05A105KA5NQNC
- C17, C18: footprint Capacitor_SMD:C_0402_1005Metric -> Capacitor_SMD:C_0603_1608Metric; LCSC C1525 -> C14663; MPN CC0402KRX7R8BB104 -> CC0603KRX7R9BB104; SKU 302010024 -> (none)
- C19, C20: value 100NF -> 22UF; footprint Capacitor_SMD:C_0402_1005Metric -> Capacitor_SMD:C_0603_1608Metric; LCSC C1525 -> C59461; MPN CC0402KRX7R8BB104 -> CL10A226MQ8NRNC; SKU 302010024 -> (none)
- C21: value 100NF -> 1uF; LCSC C1525 -> C52923; MPN CC0402KRX7R8BB104 -> CL05A105KA5NQNC; SKU 302010024 -> (none)
- C22: value 100NF -> 220nF; footprint Capacitor_SMD:C_0402_1005Metric -> Capacitor_SMD:C_0603_1608Metric; LCSC C1525 -> C21120; MPN CC0402KRX7R8BB104 -> CL10B224KA8NNNC; SKU 302010024 -> (none)
- C23: value 2.2UF -> 220nF; LCSC C23630 -> C21120; MPN EMK107BJ225KA-T -> CL10B224KA8NNNC; SKU 302010233 -> (none)
- C24: value 470pF -> 1uF; LCSC C1537 -> C52923; MPN 0402B471K500NT -> CL05A105KA5NQNC; Tempo GRM155R71H471KA01D -> (none)
- C25, C26: value 470pF -> 220nF; footprint Capacitor_SMD:C_0402_1005Metric -> Capacitor_SMD:C_0603_1608Metric; LCSC C1537 -> C21120; MPN 0402B471K500NT -> CL10B224KA8NNNC; Tempo GRM155R71H471KA01D -> (none)
- C27: value 470pF -> 1NF; LCSC C1537 -> C1523; MPN 0402B471K500NT -> 0402B102K500NT; Tempo GRM155R71H471KA01D -> (none)
- J3: footprint Connector_JST:JST_PH_B2B-PH-SM4-TB_1x02-1MP_P2.00mm_Vertical -> Connector_JST:JST_PH_B2B-PH-K_1x02_P2.00mm_Vertical; symbol Connector_Generic:Conn_01x02 -> kevin:Speaker; Link https://www.newark.com/jst-japan-solderless-terminals/b2b-p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 -> (none); MPN B2B-PH-SM4-TB(LF)(SN) -> B2B-PH-K-S(LF)(SN); Vendor Newark -> (none)
- J4: footprint Connector_JST:JST_PH_B2B-PH-SM4-TB_1x02-1MP_P2.00mm_Vertical -> Connector_JST:JST_PH_B2B-PH-K_1x02_P2.00mm_Vertical; symbol Connector_Generic:Conn_01x02 -> kevin:Speaker; Link https://www.newark.com/jst-japan-solderless-terminals/b2b-p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 -> (none); MPN B2B-PH-SM4-TB(LF)(SN) -> B2B-PH-K-S(LF)(SN)
- R47: value 10k -> 0R; LCSC C25744 -> C17168; MPN RC0402FR-0710KL -> 0402WGF0000TCE
- R56: value 0R -> 0R - DNP; footprint Resistor_SMD:R_1206_3216Metric -> Resistor_SMD:R_0402_1005Metric; LCSC C17888 -> C17168-DNP; MPN 1206W4F0000T5E -> DNP-0402WGF0000TCE; Tempo RK73Z2BTTD -> (none)
- R6: value 220k -> 120k; LCSC C25767 -> C25750; MPN 0402WGF2203TCE -> 0402WGF1203TCE; Tempo ERJ-2GEJ224X -> (none)
- R7: value 220k -> 0R; footprint Resistor_SMD:R_0402_1005Metric -> Resistor_SMD:R_0603_1608Metric; LCSC C25767 -> C21189; MPN 0402WGF2203TCE -> 0603WAF0000T5E; Tempo ERJ-2GEJ224X -> RC0603JR-070RL
Connections:
- net labels added: AVDD, DVDD, I2S_BCLK_AMP, I2S_BCLK_PI, I2S_BCLK_XMOS, I2S_DIN_AMP, I2S_DIN_PI, I2S_DOUT_PI, I2S_DOUT_XMOS, I2S_LRCK_AMP, I2S_LRCK_PI, I2S_LRCK_XMOS, I2S_MCLK_PI, I2S_MCLK_XMOS, Left+, Left-, OUT_A1+, OUT_A1-, OUT_B1+, OUT_B1-, Right+, Right-, SDOUT_I2S_AMP, VR_DIG
- net labels removed: ADDR1_3V3, ADDR2_3V3, GNDA, GPIO4, I2S_BCK, I2S_BCLK, I2S_DATA, I2S_DIN, I2S_DOUT, I2S_LRCK, I2S_SCK, MCLK, MUTE, PGND, SYNCOUT
- wire segments 221 -> 148
- no-connect marks 0 -> 3
Other:
- note added: "1.5V Digital"
- note added: "5.0V Analog"
- note added: "Address:\n0x58 - 4.7k\n0x5A - 15k \n0x5C - 47k \n0x5E - 120k"
- note added: "Ferrite Beads 300 ohm/3A"
- note added: "I2S Selector & Buffer"
- note added: "PVDD: 4.5-26.4V\nDVDD: 3.3V\nTemp: -25 to 85C\n23 Watt Max - 1.6amp"
- note added: "USB Option\nPopulate R52, R56, R63\nDNP R16, R47, R53, R62, R66\n"
- note removed: "Audio Amp & USB Sound Card"
- note removed: "Change part to \nTAS5711PHPR"
- note removed: "Ferrites 100-600 ohm/3A"
- note removed: "I2S Data from \nUSB Soundcard"
- note removed: "I2S to Line Out"
- note removed: "PGND"
- note removed: "PVDD: 4.5-14V\nVDD: 3-3.6V\nTemp: -40 to 85C\n20 Watt Max - 1.6amp"
- note removed: "Reference Diagram"
- note removed: "TODO: Add in LINE IN for testing purposes\nTODO: LINE OUT"
- note removed: "https://learn.adafruit.com/assets/48419"
- note removed: "i2c Addr is 0x4B"
- moved on the sheet: C17, C61, FB1, FB2, FB3, FB4, R25, R37, R48, R49, R50, R54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

Commit message: Rev4 Update - fix some wiring, export for printing Rev 4
Parts:
- removed J9: AudioJack3_Ground_Switch, mycroft:STX-3790-5N, symbol Connector:AudioJack2_Ground_Switch
- removed R56: 0R - DNP, Resistor_SMD:R_0402_1005Metric, symbol Device:R_Small
- added J2: AudioJack2_Ground, user:Jack_3.5mm_PJ-3210, symbol Connector:AudioJack2_Ground
- added R33: 0R, Resistor_SMD:R_0402_1005Metric, symbol Device:R_Small
Connections:
- wire segments 148 -> 146
Changed lines of the file:
@@
 Sheet 3 7
 Title ""
-Date "2020-11-18"
-Rev "rev4 - 0.01"
+Date "2020-11-22"
+Rev "Rev4 - 0.03"
 Comp "Mycroft"
-Comment1 "SJ201 r4.01"
+Comment1 "SJ-201-R4"
 Comment2 ""
 Comment3 ""
@@
 Text GLabel 5350 1550 2    51   Input ~ 0
 PVDD
-$Comp
-L Connector:AudioJack2_Ground_Switch J9
-U 1 1 5FDDA9C6
-P 6125 4475
-F 0 "J9" H 6107 4900 50  0000 C CNN
-F 1 "AudioJack3_Ground_Switch" H 6107 4809 50  0000 C CNN
-F 2 "mycroft:STX-3790-5N" H 6125 4475 50  0001 C CNN
-F 3 "~" H 6125 4475 50  0001 C CNN
-F 4 "DNP " H 6125 4475 50  0001 C CNN "MPN"
-F 5 "2092-STX-3790-5N-ND" H 6125 4475 50  0001 C CNN "Digikey"
-F 6 "https://www.digikey.com/product-detail/en/kycon-inc/STX-3790-5N/2092-STX-3790-5N-ND/9990125" H 6125 4475 50  0001 C CNN "Link"
-	1    6125 4475
-	1    0    0    -1
-$EndComp
-$Comp
-L power:GND #PWR0117
-U 1 1 5FDDB40B
-P 6125 4775
-F 0 "#PWR0117" H 6125 4525 50  0001 C CNN
-F 1 "GND" H 6130 4602 50  0000 C CNN
-F 2 "" H 6125 4775 50  0001 C CNN
-F 3 "" H 6125 4775 50  0001 C CNN
-	1    6125 4775
-	1    0    0    -1
-$EndComp
-Text GLabel 6325 4575 2    51   Input ~ 0
-VoutL
-Text GLabel 6325 4375 2    51   Input ~ 0
-VoutR
-Wire Wire Line
-	6325 4375 6325 4275
-Wire Wire Line
-	6325 4475 6325 4575
 Text GLabel 7450 5975 3    51   Input ~ 0
 SDA
@@
 $Comp
 L Device:R_Small R?
-U 1 1 5FF12B3D
-P 1700 7125
-AR Path="/5EA9C461/5FF12B3D" Ref="R?"  Part="1"
-AR Path="/5EA9C67D/5FF12B3D" Ref="R56"  Part="1"
-AR Path="/5EA9C76D/5FF12B3D" Ref="R?"  Part="1"
-F 0 "R56" V 1650 6900 50  0000 L CNN
-F 1 "0R - DNP" V 1750 7225 50  0000 L CNN
-F 2 "Resistor_SMD:R_0402_1005Metric" H 1700 7125 50  0001 C CNN
-F 3 "~" H 1700 7125 50  0001 C CNN
-F 4 "DNP-0402WGF0000TCE" H 1700 7125 50  0001 C CNN "MPN"
-F 5 "C17168-DNP" H 1700 7125 50  0001 C CNN "LCSC"
-	1    1700 7125
-	0    1    1    0
-$EndComp
-$Comp
-L Device:R_Small R?
 U 1 1 5FF12EBA
 P 3275 7475
@@
 $EndComp
 Connection ~ 2250 7125
+$Comp
+L Connector:AudioJack2_Ground J2
+U 1 1 60817512
+P 7075 4500
+F 0 "J2" H 7107 4825 50  0000 C CNN
+F 1 "AudioJack2_Ground" H 7107 4734 50  0000 C CNN
+F 2 "user:Jack_3.5mm_PJ-3210" H 7075 4500 50  0001 C CNN
+F 3 "~" H 7075 4500 50  0001 C CNN
+F 4 "PJ-3210-4A" H 7075 4500 50  0001 C CNN "MPN"
+F 5 "C136686" H 7075 4500 50  0001 C CNN "LCSC"
+F 6 "https://lcsc.com/product-detail/Audio-Video-Connectors_Korean-Hroparts-Elec-PJ-3210-4A_C136686.html" H 7075 4500 50  0001 C CNN "Link"
+	1    7075 4500
+	1    0    0    -1
+$EndComp
+Text GLabel 7275 4400 2    51   Input ~ 0
+VoutR
+Text GLabel 7275 4500 2    51   Input ~ 0
+VoutL
+$Comp
+L power:GND #PWR0149
+U 1 1 60817CE6
+P 7075 4700
+F 0 "#PWR0149" H 7075 4450 50  0001 C CNN
+F 1 "GND" H 7080 4527 50  0000 C CNN
+F 2 "" H 7075 4700 50  0001 C CNN
+F 3 "" H 7075 4700 50  0001 C CNN
+	1    7075 4700
+	1    0    0    -1
+$EndComp
+$Comp
+L Device:R_Small R?
+U 1 1 60AD536C
+P 1700 7125
+AR Path="/5EA9C461/60AD536C" Ref="R?"  Part="1"
+AR Path="/5EA9C67D/60AD536C" Ref="R33"  Part="1"
+AR Path="/5EA9C76D/60AD536C" Ref="R?"  Part="1"
+F 0 "R33" V 1650 6900 50  0000 L CNN
+F 1 "0R" V 1750 7225 50  0000 L CNN
+F 2 "Resistor_SMD:R_0402_1005Metric" H 1700 7125 50  0001 C CNN
+F 3 "~" H 1700 7125 50  0001 C CNN
+F 4 "0402WGF0000TCE" H 1700 7125 50  0001 C CNN "MPN"
+F 5 "C17168" H 1700 7125 50  0001 C CNN "LCSC"
+	1    1700 7125
+	0    1    1    0
+$EndComp
 $EndSCHEMATC

Commit message: SJ-201-R6 for FAB - removed buffer IC
Parts:
- removed R25, R37: 0R - DNP, Resistor_SMD:R_0603_1608Metric, symbol Device:R_Small
- removed R47, R53, R62: 0R, Resistor_SMD:R_0402_1005Metric, symbol Device:R_Small
- removed R52, R63: 0R - DNP, Resistor_SMD:R_0402_1005Metric, symbol Device:R_Small
- removed R54, R55: 0R, Resistor_SMD:R_0603_1608Metric, symbol Device:R_Small
- removed U14: NC7NZ34K8XTR, NC7N:ON_Semi-NZ34-0-0-0, symbol nc7nz:NC7NZ34K8X
- added C29, C30: 1uF, Capacitor_SMD:C_0402_1005Metric, symbol Device:C_Small
- added C70: 100NF, Capacitor_SMD:C_0402_1005Metric, symbol Device:C_Small
- added C73: 10UF, Capacitor_SMD:C_0402_1005Metric, symbol Device:C_Small
- added C74, C75: 10nF, Capacitor_SMD:C_0402_1005Metric, symbol Device:C_Small
- added FB7: FB, Resistor_SMD:R_1206_3216Metric, symbol kevin:Ferrite_Bead_Small
- added NT1: Net-Tie_2, NetTie:NetTie-2_SMD_Pad0.5mm, symbol Device:Net-Tie_2
- added OutL1, OutR1: TestPoint, TestPoint:TestPoint_Pad_D2.0mm, symbol Connector:TestPoint
- added R31: 33R, Resistor_SMD:R_0402_1005Metric, symbol Device:R_Small
- added R61, R67: 220k, Resistor_SMD:R_0402_1005Metric, symbol Device:R_Small
- added R68, R69: 100R, Resistor_SMD:R_0402_1005Metric, symbol Device:R_Small
- added U16: UDA1334ATS, Package_SO:SSOP-16_4.4x5.2mm_P0.65mm, symbol Audio:UDA1334ATS
- J3, J4: LCSC (none) -> C131337
- R16, R33: value 0R -> 33R; LCSC C17168 -> C25105; MPN 0402WGF0000TCE -> 0402WGF330JTCE; Tempo (none) -> RC0402FR-0733RL
- TP1, TP3, TP4: footprint TestPoint:TestPoint_Pad_D1.0mm -> TestPoint:TestPoint_Pad_D2.0mm
- U3: Link (none) -> https://www.mouser.com/ProductDetail/Texas-Instruments/TAS5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
Connections:
- net labels added: I2S_BCLK_UDA, I2S_DIN_XMOS, I2S_LRCK_UDA, I2S_WS_PI, PGND, TAS_Fault, UDA_L, UDA_R
- net labels removed: I2S_LRCK_PI
- wire segments 146 -> 189
- no-connect marks 3 -> 1
Other:
- note added: "Address:\n0x58 - 4.7k\n0x5A - 15k \n0x5C - 47k \n0x5E - 120k - 0x2F actual"
- note added: "I2C Route"
- note added: "I2S Selector"
- note removed: "Address:\n0x58 - 4.7k\n0x5A - 15k \n0x5C - 47k \n0x5E - 120k"
- note removed: "I2C Selector"
- note removed: "I2C Selector\nPopulate:\nR54 and R55 for Raspi\nR25 and R37 for XMOS"
- note removed: "I2S Selector & Buffer"
- note removed: "USB Option\nPopulate R52, R56, R63\nDNP R16, R47, R53, R62, R66\n"
- moved on the sheet: C10, C11, C12, C13, C14, C15, C16, C17, C18, C19, C20, C21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

Commit message: Removed unused files, cleaned up directory, remove SJ202
Parts:
- J2: footprint user:Jack_3.5mm_PJ-3210 -> Mycroft:Jack_3.5mm_PJ-3210
Changed lines of the file:
@@
 F 0 "J2" H 9675 4700 50  0000 C CNN
 F 1 "AudioJack2_Ground" H 9275 4250 50  0000 C CNN
-F 2 "user:Jack_3.5mm_PJ-3210" H 9750 4475 50  0001 C CNN
+F 2 "Mycroft:Jack_3.5mm_PJ-3210" H 9750 4475 50  0001 C CNN
 F 3 "~" H 9750 4475 50  0001 C CNN
 F 4 "PJ-3210-4A" H 9750 4475 50  0001 C CNN "MPN"

Commit message: Update libraries, reorganize files
Parts:
- FB1, FB2, FB3, FB4, FB7: symbol kevin:Ferrite_Bead_Small -> Mycroft:Ferrite_Bead_Small
- J3, J4: symbol kevin:Speaker -> Mycroft:Speaker
Changed lines of the file:
@@
 $EndComp
 $Comp
-L kevin:Speaker J4
+L Mycroft:Speaker J4
 U 1 1 5F1C4478
 P 8075 2475
+AR Path="/5F1C4478" Ref="J4"  Part="1"
+AR Path="/5EA9C67D/5F1C4478" Ref="J4"  Part="1"
 F 0 "J4" H 8275 2350 50  0000 C CNN
 F 1 "SPK" H 8300 2525 50  0000 C CNN
@@
 $EndComp
 $Comp
-L kevin:Speaker J3
+L Mycroft:Speaker J3
 U 1 1 5F17E7BB
 P 8075 1475
+AR Path="/5F17E7BB" Ref="J3"  Part="1"
+AR Path="/5EA9C67D/5F17E7BB" Ref="J3"  Part="1"
 F 0 "J3" H 8225 1450 50  0000 L CNN
 F 1 "SPK" H 8225 1300 50  0000 L CNN
@@
 Connection ~ 6100 2075
 $Comp
-L kevin:Ferrite_Bead_Small FB?
+L Mycroft:Ferrite_Bead_Small FB?
 U 1 1 5F093200
 P 6575 1225
@@
 AR Path="/5EAB86B0/5F093200" Ref="FB?"  Part="1"
 AR Path="/5EA9C67D/5F093200" Ref="FB1"  Part="1"
+AR Path="/5F093200" Ref="FB1"  Part="1"
 F 0 "FB1" V 6525 1125 50  0000 C CNN
 F 1 "FB" V 6700 1325 50  0000 C CNN
@@
 $EndComp
 $Comp
-L kevin:Ferrite_Bead_Small FB?
+L Mycroft:Ferrite_Bead_Small FB?
 U 1 1 5F1C4447
 P 6575 2775
@@
 AR Path="/5EAB86B0/5F1C4447" Ref="FB?"  Part="1"
 AR Path="/5EA9C67D/5F1C4447" Ref="FB4"  Part="1"
+AR Path="/5F1C4447" Ref="FB4"  Part="1"
 F 0 "FB4" V 6525 2675 50  0000 C CNN
 F 1 "FB" V 6625 2875 50  0000 C CNN
@@
 $EndComp
 $Comp
-L kevin:Ferrite_Bead_Small FB?
+L Mycroft:Ferrite_Bead_Small FB?
 U 1 1 5F1C4441
 P 6575 2200
@@
 AR Path="/5EAB86B0/5F1C4441" Ref="FB?"  Part="1"
 AR Path="/5EA9C67D/5F1C4441" Ref="FB3"  Part="1"
+AR Path="/5F1C4441" Ref="FB3"  Part="1"
 F 0 "FB3" V 6525 2100 50  0000 C CNN
 F 1 "FB" V 6700 2300 50  0000 C CNN
@@
 $EndComp
 $Comp
-L kevin:Ferrite_Bead_Small FB?
+L Mycroft:Ferrite_Bead_Small FB?
 U 1 1 5F093B93
 P 6575 1675
@@
 AR Path="/5EAB86B0/5F093B93" Ref="FB?"  Part="1"
 AR Path="/5EA9C67D/5F093B93" Ref="FB2"  Part="1"
+AR Path="/5F093B93" Ref="FB2"  Part="1"
 F 0 "FB2" V 6525 1575 50  0000 C CNN
 F 1 "FB" V 6625 1775 50  0000 C CNN
@@
 	8425 3675 8700 3675
 $Comp
-L kevin:Ferrite_Bead_Small FB?
+L Mycroft:Ferrite_Bead_Small FB?
 U 1 1 5FD80208
 P 8225 3100
@@
 AR Path="/5EAB86B0/5FD80208" Ref="FB?"  Part="1"
 AR Path="/5EA9C67D/5FD80208" Ref="FB7"  Part="1"
+AR Path="/5FD80208" Ref="FB7"  Part="1"
 F 0 "FB7" V 8175 3000 50  0000 C CNN
 F 1 "FB" V 8350 3200 50  0000 C CNN
