File: mark-II-Rpi-devkit/KiCAD/SJ201-Raspberry Pi 4 Daughterboard/Power.sch (KiCad schematic (older format))
At the start: 37 parts, among them J1 Barrel_Jack, J12 GND, J5 PowerTP, Q3 AO3415A, U1 XL4501E1, U2 NCP303LSN09, U4 AZ1117CH-3.3, U7 MP2359

Commit message: Fix missing items in schematic in Github
Parts:
- C2, C5, C7, C8, C9: symbol OPL_Capacitor:CERAMIC-2.2UF-25V-10%-X7R_0805_ -> Device:C_Small
- C3, C4, C63: symbol OPL_Capacitor:CERAMIC-100NF-50V-10%-X7R_0805_ -> Device:C_Small
- L2: symbol OPL_Inductor:SMD-INDUCTOR-2.2UH-20%-1.2A_0805_ -> Device:L
Changed lines of the file:
@@
 AR Path="/5EA9C76D/5F710DF7" Ref="R?"  Part="1"
 AR Path="/5EAAC9A5/5F710DF7" Ref="R8"  Part="1"
-F 0 "R8" H 5300 3500 50  0000 L CNN
-F 1 "3.3K" H 5250 3575 50  0000 L CNN
+F 0 "R8" H 5325 3500 50  0000 L CNN
+F 1 "3.3K" H 5250 3600 50  0000 L CNN
 F 2 "Resistor_SMD:R_0402_1005Metric" H 5475 3525 50  0001 C CNN
 F 3 "~" H 5475 3525 50  0001 C CNN
@@
 	1    0    0    -1
 $EndComp
-Wire Wire Line
-	4525 3275 4525 3075
 $Comp
-L OPL_Capacitor:CERAMIC-2.2UF-25V-10%-X7R_0805_ C8
+L Device:C_Small C8
 U 1 1 5F2A4E27
 P 5825 3225
-F 0 "C8" V 5783 3293 45  0000 L CNN
-F 1 "33NF" V 5867 3293 45  0000 L CNN
+F 0 "C8" H 5900 3300 45  0000 L CNN
+F 1 "33NF" H 5900 3125 45  0000 L CNN
 F 2 "Capacitor_SMD:C_0402_1005Metric" H 5825 3225 50  0001 C CNN
 F 3 "" H 5825 3225 50  0001 C CNN
@@
 F 6 "508000001" H 5825 3225 50  0001 C CNN "SKU"
 	1    5825 3225
-	0    1    1    0
+	1    0    0    -1
 $EndComp
 Wire Wire Line
@@
 AR Path="/5EA9C461/5F2B6A94" Ref="C?"  Part="1"
 AR Path="/5EAAC9A5/5F2B6A94" Ref="C60"  Part="1"
-F 0 "C60" H 2600 4950 45  0000 R CNN
-F 1 "22UF" H 2625 4875 45  0000 R CNN
+F 0 "C60" H 2525 4975 45  0000 R CNN
+F 1 "22UF" H 2575 4825 45  0000 R CNN
 F 2 "Capacitor_SMD:C_0603_1608Metric" H 2350 4900 50  0001 C CNN
 F 3 "" H 2350 4900 50  0001 C CNN
@@
 AR Path="/5EA9C76D/5EFB61C2" Ref="R?"  Part="1"
 AR Path="/5EAAC9A5/5EFB61C2" Ref="R28"  Part="1"
-F 0 "R28" H 6425 3150 50  0000 L CNN
-F 1 "680R" H 6375 3225 50  0000 L CNN
+F 0 "R28" H 6450 3125 50  0000 L CNN
+F 1 "680R" H 6400 3225 50  0000 L CNN
 F 2 "Resistor_SMD:R_0402_1005Metric" H 6650 3175 50  0001 C CNN
 F 3 "~" H 6650 3175 50  0001 C CNN
@@
 	8250 1175 8100 1175
 $Comp
-L OPL_Capacitor:CERAMIC-100NF-50V-10%-X7R_0805_ C?
+L Device:C_Small C?
 U 1 1 5F36D909
 P 8100 1325
 AR Path="/5EA9C76D/5F36D909" Ref="C?"  Part="1"
 AR Path="/5EAAC9A5/5F36D909" Ref="C63"  Part="1"
-F 0 "C63" V 8058 1393 45  0000 L CNN
-F 1 "100NF" V 8142 1393 45  0000 L CNN
+F 0 "C63" H 8150 1400 45  0000 L CNN
+F 1 "100NF" H 8125 1250 45  0000 L CNN
 F 2 "Capacitor_SMD:C_0402_1005Metric" H 8100 1325 50  0001 C CNN
 F 3 "" H 8100 1325 50  0001 C CNN
@@
 F 6 "C1525" H 8100 1325 50  0001 C CNN "LCSC"
 	1    8100 1325
-	0    1    1    0
+	1    0    0    -1
 $EndComp
 $Comp
@@
 	0    1    1    0
 $EndComp
-$Comp
-L OPL_Capacitor:CERAMIC-100NF-50V-10%-X7R_0805_ C?
-U 1 1 5F0D59F2
-P 4525 3425
-AR Path="/5EA9C76D/5F0D59F2" Ref="C?"  Part="1"
-AR Path="/5EAAC9A5/5F0D59F2" Ref="C4"  Part="1"
-F 0 "C4" V 4483 3493 45  0000 L CNN
-F 1 "1uF" V 4567 3493 45  0000 L CNN
-F 2 "Capacitor_SMD:C_0402_1005Metric" H 4525 3425 50  0001 C CNN
-F 3 "" H 4525 3425 50  0001 C CNN
-F 4 "CC0402KRX5R6BB105" H 4555 3575 20  0001 C CNN "MPN"
-F 5 "302010040" H 4555 3575 20  0001 C CNN "SKU"
-F 6 "C52923" H 4525 3425 50  0001 C CNN "LCSC"
-	1    4525 3425
-	0    1    1    0
-$EndComp
 Connection ~ 4525 3075
 Wire Wire Line
@@
 Wire Wire Line
 	3900 3600 3900 3400
-Connection ~ 5825 3075
-Wire Wire Line
-	5825 3075 6200 3075
 Wire Wire Line
 	4525 3075 4850 3075
@@
 	5475 3125 5475 3075
 Connection ~ 5475 3075
-Wire Wire Line
-	5475 3075 5825 3075
 $Comp
 L power:GND #PWR06
@@
 	2825 3275 2825 3400
 $Comp
-L OPL_Capacitor:CERAMIC-100NF-50V-10%-X7R_0805_ C?
+L Device:C_Small C?
 U 1 1 5F0EF382
 P 2175 3225
 AR Path="/5EA9C76D/5F0EF382" Ref="C?"  Part="1"
 AR Path="/5EAAC9A5/5F0EF382" Ref="C3"  Part="1"
-F 0 "C3" V 2133 3293 45  0000 L CNN
-F 1 "1uF" V 2217 3293 45  0000 L CNN
+F 0 "C3" H 2025 3300 45  0000 L CNN
+F 1 "1uF" H 1975 3150 45  0000 L CNN
 F 2 "Capacitor_SMD:C_0402_1005Metric" H 2175 3225 50  0001 C CNN
 F 3 "" H 2175 3225 50  0001 C CNN
@@
 F 6 "C52923" H 2175 3225 50  0001 C CNN "LCSC"
 	1    2175 3225
-	0    1    1    0
+	-1   0    0    -1
 $EndComp
-Connection ~ 2175 3075
-Wire Wire Line
-	2175 3075 1600 3075
-Wire Wire Line
-	2175 3375 2175 3675
 Wire Wire Line
 	2175 3675 1600 3675
@@
 VFB = 0.6V\nVO  = 0.6 x (1 + 30/47) = 0.98V\n
 $Comp
-L OPL_Inductor:SMD-INDUCTOR-2.2UH-20%-1.2A_0805_ L?
+L Device:L L?
 U 1 1 5F44B395
 P 3825 6550
 AR Path="/5EA9C76D/5F44B395" Ref="L?"  Part="1"
 AR Path="/5EAAC9A5/5F44B395" Ref="L2"  Part="1"
-F 0 "L2" H 3825 6729 45  0000 C CNN
-F 1 "2.2UH ±30% 1.55A" H 3825 6645 45  0000 C CNN
+F 0 "L2" V 3950 6550 45  0000 C CNN
+F 1 "2.2UH ±30% 1.55A" V 3900 6450 45  0000 C CNN
 F 2 "Inductor_SMD:L_1210_3225Metric" H 3825 6550 60  0001 C CNN
 F 3 "https://datasheet.lcsc.com/szlcsc/Murata-Electronics-LQH32PN2R2NN0L_C86074.pdf" H 3825 6550 60  0001 C CNN
@@
 F 5 "LQH32PN2R2NN0L" H 3825 6550 50  0001 C CNN "MPN"
 	1    3825 6550
-	1    0    0    -1
+	0    -1   -1   0
 $EndComp
 $Comp
-L OPL_Capacitor:CERAMIC-2.2UF-25V-10%-X7R_0805_ C?
+L Device:C_Small C?
 U 1 1 5F44B39E
 P 1650 6450
 AR Path="/5EA9C76D/5F44B39E" Ref="C?"  Part="1"
 AR Path="/5EAAC9A5/5F44B39E" Ref="C5"  Part="1"
-F 0 "C5" V 1692 6382 45  0000 R CNN
-F 1 "10UF" V 1608 6382 45  0000 R CNN
+F 0 "C5" H 1575 6375 45  0000 R CNN
+F 1 "10UF" H 1600 6525 45  0000 R CNN
 F 2 "Capacitor_SMD:C_0402_1005Metric" H 1650 6450 50  0001 C CNN
 F 3 "" H 1650 6450 50  0001 C CNN
@@
 F 6 "C15525" H 1650 6450 50  0001 C CNN "LCSC"
 	1    1650 6450
-	0    -1   -1   0
+	-1   0    0    1
 $EndComp
-Wire Wire Line
-	4025 6550 4325 6550
 $Comp
 L power:+5V #PWR010
@@
 AR Path="/5EA9C461/5F44C846" Ref="C?"  Part="1"
 AR Path="/5EAAC9A5/5F44C846" Ref="C37"  Part="1"
-F 0 "C37" H 4950 6800 45  0000 R CNN
-F 1 "22UF" H 4975 6725 45  0000 R CNN
+F 0 "C37" H 4900 6825 45  0000 R CNN
+F 1 "22UF" H 4950 6675 45  0000 R CNN
 F 2 "Capacitor_SMD:C_0603_1608Metric" H 4700 6750 50  0001 C CNN
 F 3 "" H 4700 6750 50  0001 C CNN
@@
 $EndComp
 $Comp
-L OPL_Capacitor:CERAMIC-2.2UF-25V-10%-X7R_0805_ C?
+L Device:C_Small C?
 U 1 1 5F45B365
 P 3250 6350
 AR Path="/5EA9C76D/5F45B365" Ref="C?"  Part="1"
 AR Path="/5EAAC9A5/5F45B365" Ref="C7"  Part="1"
-F 0 "C7" V 3292 6282 45  0000 R CNN
-F 1 "10nF" V 3208 6282 45  0000 R CNN
+F 0 "C7" H 3175 6275 45  0000 R CNN
+F 1 "10nF" H 3175 6425 45  0000 R CNN
 F 2 "Capacitor_SMD:C_0402_1005Metric" H 3250 6350 50  0001 C CNN
 F 3 "" H 3250 6350 50  0001 C CNN
 F 4 "C15195" H 3250 6350 50  0001 C CNN "LCSC"
 	1    3250 6350
-	0    -1   -1   0
+	-1   0    0    1
 $EndComp
 $Comp
@@
 	3250 6500 3150 6500
 Wire Wire Line
-	3625 6550 3400 6550
-Wire Wire Line
 	3250 6500 3250 6550
 Wire Wire Line
 	3250 6550 3400 6550
-Connection ~ 3250 6500
 Connection ~ 3400 6550
 $Comp
@@
 Wire Wire Line
 	4325 6875 4325 6950
-Wire Wire Line
-	1650 6200 1650 6300
 Connection ~ 1650 6200
-Wire Wire Line
-	1650 6750 1650 6600
 Text Notes 4125 1075 0    50   ~ 0
 Power Test Points
@@
 EndData
 $EndBitmap
-Wire Wire Line
-	2175 3075 2825 3075
 $Comp
 L power:GND #PWR0157
@@
 $EndComp
 $Comp
-L OPL_Capacitor:CERAMIC-2.2UF-25V-10%-X7R_0805_ C2
+L Device:C_Small C2
 U 1 1 5F3AC2DA
 P 3350 5200
 AR Path="/5EAAC9A5/5F3AC2DA" Ref="C2"  Part="1"
 AR Path="/5EA9C76D/5F3AC2DA" Ref="C?"  Part="1"
-F 0 "C2" V 3308 5268 45  0000 L CNN
-F 1 "2.2NF" V 3392 5268 45  0000 L CNN
+F 0 "C2" H 3200 5250 45  0000 L CNN
+F 1 "2.2NF" H 3100 5125 45  0000 L CNN
 F 2 "Capacitor_SMD:C_0402_1005Metric" H 3350 5200 50  0001 C CNN
 F 3 "https://statics3.seeedstudio.com/images/opl/datasheet/302010022.pdf" H 3350 5200 50  0001 C CNN
@@
 F 6 "C1531" H 3350 5200 50  0001 C CNN "LCSC"
 	1    3350 5200
-	0    1    1    0
+	-1   0    0    -1
 $EndComp
 $Comp
@@
 	4775 4900 4725 4900
 $Comp
-L OPL_Capacitor:CERAMIC-2.2UF-25V-10%-X7R_0805_ C9
+L Device:C_Small C9
 U 1 1 5F3AC2F9
 P 4975 5075
 AR Path="/5EAAC9A5/5F3AC2F9" Ref="C9"  Part="1"
 AR Path="/5EA9C76D/5F3AC2F9" Ref="C?"  Part="1"
-F 0 "C9" V 4933 5143 45  0000 L CNN
-F 1 "1NF" V 5017 5143 45  0000 L CNN
+F 0 "C9" H 4825 5000 45  0000 L CNN
+F 1 "1NF" H 4775 5150 45  0000 L CNN
 F 2 "Capacitor_SMD:C_0402_1005Metric" H 4975 5075 50  0001 C CNN
 F 3 "https://statics3.seeedstudio.com/images/opl/datasheet/302010005.pdf" H 4975 5075 50  0001 C CNN
@@
 F 6 "C1523" H 4975 5075 50  0001 C CNN "LCSC"
 	1    4975 5075
-	0    1    1    0
+	1    0    0    -1
 $EndComp
 $Comp
@@
 Wire Wire Line
 	4775 4900 4975 4900
-Wire Wire Line
-	4975 4900 4975 4925
 Connection ~ 4775 4900
 Wire Notes Line
@@
 Wire Notes Line
 	3750 950  3750 2125
+Wire Wire Line
+	8100 1225 8100 1175
+Wire Wire Line
+	8100 1425 8100 1475
+Wire Wire Line
+	3350 5100 3350 5050
+Wire Wire Line
+	3350 5300 3350 5350
+Wire Wire Line
+	4975 4900 4975 4975
+Wire Wire Line
+	4975 5175 4975 5225
+Wire Wire Line
+	5475 3075 5825 3075
+Wire Wire Line
+	1600 3075 2175 3075
+Wire Wire Line
+	4525 3575 4525 3525
+Wire Wire Line
+	4525 3075 4525 3325
+$Comp
+L Device:C_Small C?
+U 1 1 5F0D59F2
+P 4525 3425
+AR Path="/5EA9C76D/5F0D59F2" Ref="C?"  Part="1"
+AR Path="/5EAAC9A5/5F0D59F2" Ref="C4"  Part="1"
+F 0 "C4" H 4375 3500 45  0000 L CNN
+F 1 "1uF" H 4350 3350 45  0000 L CNN
+F 2 "Capacitor_SMD:C_0402_1005Metric" H 4525 3425 50  0001 C CNN
+F 3 "" H 4525 3425 50  0001 C CNN
+F 4 "CC0402KRX5R6BB105" H 4555 3575 20  0001 C CNN "MPN"
+F 5 "302010040" H 4555 3575 20  0001 C CNN "SKU"
+F 6 "C52923" H 4525 3425 50  0001 C CNN "LCSC"
+	1    4525 3425
+	-1   0    0    -1
+$EndComp
+Wire Wire Line
+	2175 3125 2175 3075
+Connection ~ 2175 3075
+Wire Wire Line
+	2175 3075 2825 3075
+Wire Wire Line
+	2175 3325 2175 3675
+Wire Wire Line
+	3250 6500 3250 6450
+Connection ~ 3250 6500
+Wire Wire Line
+	3250 6250 3250 6200
+Wire Wire Line
+	5825 3125 5825 3075
+Connection ~ 5825 3075
+Wire Wire Line
+	5825 3075 6200 3075
+Wire Wire Line
+	5825 3325 5825 3375
+Wire Wire Line
+	3400 6550 3675 6550
+Wire Wire Line
+	3975 6550 4325 6550
+Wire Wire Line
+	1650 6550 1650 6750
+Wire Wire Line
+	1650 6200 1650 6350
 $EndSCHEMATC

Commit message: SJ201 - Removed CM108b soundcard, added in I2S to Line out, ATTin402. Moved holes in layout. SJ202 - extened length to plug into USB2.0 port
Parts:
- removed J12: GND, Connector_PinHeader_2.54mm:PinHeader_1x02_P2.54mm_Vertical, symbol Connector_Generic:Conn_01x02
- C1: Link (none) -> https://lcsc.com/product-detail/Aluminum-Electrolytic-Capac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; Vendor (none) -> LCSC
- C2: Link (none) -> https://lcsc.com/product-detail/Multilayer-Ceramic-Capacito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; MPN CC0402KRX7R9BB222 -> 0402B222K500NT; SKU 302010022 -> (none); Vendor (none) -> LCSC
- C3, C4: MPN CC0402KRX5R6BB105 -> CL05A105KA5NQNC; SKU 302010040 -> (none)
- C7: MPN (none) -> CL05B103KB5NNNC
- J5: footprint Connector_PinHeader_2.54mm:PinHeader_2x03_P2.54mm_Vertical -> Connector_PinHeader_2.54mm:PinHeader_2x04_P2.54mm_Vertical; symbol Connector_Generic:Conn_02x03_Odd_Even -> Connector_Generic:Conn_02x04_Odd_Even; MPN (none) -> DNP
- L1: Link (none) -> https://lcsc.com/product-detail/Power-Inductors_TDG-TMAX-13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
- PWR1: value LED -> LED_RED
- Q3: value AO3415A -> AO3401A; footprint digikey-footprints:SOT-23-3 -> Package_TO_SOT_SMD:SOT-23; Category Discrete Semiconductor Products -> (none); DK_Datasheet_Link http://aosmd.com/res/data_sheets/AO3415A.pdf -> (none); Description MOSFET P-CH 20V 5A SOT23-3 -> (none); Digi-Key_PN 785-1193-1-ND -> (none); Digikey 785-1193-1-ND -> (none); Family Transistors - FETs, MOSFETs - Single -> (none); LCSC C133233 -> C15127; MPN AO3415A -> AO3401A; Manufacturer Alpha & Omega Semiconductor Inc. -> (none); Status Active -> (none)
- R28: MPN (none) -> 0402WGF6800TCE
- R3: MPN (none) -> 0402WGF7502TCE
- R4: MPN (none) -> 0402WGF3303TCE
- TP1_0V1, TP25: MPN (none) -> DNP
- U4: value AZ1117CH-3.3 -> AMS1117-3.3; LCSC C92102 -> C6186; MPN AZ1117CH-3.3TRG1 -> AMS1117-3.3
Connections:
- net labels added: PGND
Changed lines of the file:
@@
 Sheet 2 6
 Title "Power"
-Date "2020-08-16"
-Rev "0.66"
+Date "2020-09-26"
+Rev "0.67b"
 Comp "Mycroft"
 Comment1 "Power Converter"
@@
 EndData
 $EndBitmap
-Text Notes 1200 1950 0    118  ~ 0
+Text Notes 1425 2150 0    118  ~ 0
 Reference Diagram
 Text GLabel 5950 1275 2    63   Input ~ 0
@@
 P 8750 1175
 F 0 "Q3" V 8875 1225 60  0000 L CNN
-F 1 "AO3415A" V 8500 1175 60  0000 L CNN
-F 2 "digikey-footprints:SOT-23-3" H 8950 1375 60  0001 L CNN
-F 3 "http://aosmd.com/res/data_sheets/AO3401A.pdf" H 8950 1475 60  0001 L CNN
-F 4 "785-1193-1-ND" H 8950 1575 60  0001 L CNN "Digi-Key_PN"
-F 5 "AO3415A" H 8950 1675 60  0001 L CNN "MPN"
-F 6 "Discrete Semiconductor Products" H 8950 1775 60  0001 L CNN "Category"
-F 7 "Transistors - FETs, MOSFETs - Single" H 8950 1875 60  0001 L CNN "Family"
-F 8 "http://aosmd.com/res/data_sheets/AO3415A.pdf" H 8950 1975 60  0001 L CNN "DK_Datasheet_Link"
+F 1 "AO3401A" V 8500 1175 60  0000 L CNN
+F 2 "Package_TO_SOT_SMD:SOT-23" H 8950 1375 60  0001 L CNN
+F 3 "" H 8950 1475 60  0001 L CNN
+F 4 "" H 8950 1575 60  0001 L CNN "Digi-Key_PN"
+F 5 "AO3401A" H 8950 1675 60  0001 L CNN "MPN"
+F 6 "" H 8950 1775 60  0001 L CNN "Category"
+F 7 "" H 8950 1875 60  0001 L CNN "Family"
+F 8 "" H 8950 1975 60  0001 L CNN "DK_Datasheet_Link"
 F 9 "" H 8950 2075 60  0001 L CNN "DK_Detail_Page"
-F 10 "MOSFET P-CH 20V 5A SOT23-3" V 7975 600 60  0000 L CNN "Description"
-F 11 "Alpha & Omega Semiconductor Inc." H 8950 2275 60  0001 L CNN "Manufacturer"
-F 12 "Active" H 8950 2375 60  0001 L CNN "Status"
-F 13 "785-1193-1-ND" H 8750 1175 50  0001 C CNN "Digikey"
-F 14 "C133233" H 8750 1175 50  0001 C CNN "LCSC"
+F 10 "" V 7975 600 60  0000 L CNN "Description"
+F 11 "" H 8950 2275 60  0001 L CNN "Manufacturer"
+F 12 "" H 8950 2375 60  0001 L CNN "Status"
+F 13 "C15127" H 8750 1175 50  0001 C CNN "LCSC"
 	1    8750 1175
 	0    -1   -1   0
@@
 F 3 "https://datasheet.lcsc.com/szlcsc/1912111437_TDG-TMAX-1365-470-M_C429835.pdf" H 4275 3075 50  0001 C CNN
 F 4 "TMAX-1365-470-M" H 4275 3075 50  0001 C CNN "MPN"
-F 5 "" V 4275 3075 50  0001 C CNN "Link"
+F 5 "https://lcsc.com/product-detail/Power-Inductors_TDG-TMAX-1365-470-M_C429835.html" V 4275 3075 50  0001 C CNN "Link"
 F 6 "C429835" H 4275 3075 50  0001 C CNN "LCSC"
 	1    4275 3075
@@
 P 1925 4750
 F 0 "U4" H 1925 4992 50  0000 C CNN
-F 1 "AZ1117CH-3.3" H 1925 4901 50  0000 C CNN
+F 1 "AMS1117-3.3" H 1925 4901 50  0000 C CNN
 F 2 "Package_TO_SOT_SMD:SOT-223-3_TabPin2" H 1925 5000 50  0001 C CIN
-F 3 "https://www.diodes.com/assets/Datasheets/AZ1117C.pdf" H 1925 4750 50  0001 C CNN
-F 4 "AZ1117CH-3.3TRG1" H 1925 4750 50  0001 C CNN "MPN"
-F 5 "C92102" H 1925 4750 50  0001 C CNN "LCSC"
+F 3 "" H 1925 4750 50  0001 C CNN
+F 4 "AMS1117-3.3" H 1925 4750 50  0001 C CNN "MPN"
+F 5 "C6186" H 1925 4750 50  0001 C CNN "LCSC"
 	1    1925 4750
 	1    0    0    -1
@@
 P 6650 3425
 F 0 "PWR1" V 6689 3307 50  0000 R CNN
-F 1 "LED" V 6598 3307 50  0000 R CNN
+F 1 "LED_RED" V 6598 3307 50  0000 R CNN
 F 2 "LED_SMD:LED_0603_1608Metric" H 6650 3425 50  0001 C CNN
 F 3 "https://datasheet.lcsc.com/szlcsc/1811141223_TOGIALED-TJ-S1608SW6TGLC2R-A5_C192315.pdf" H 6650 3425 50  0001 C CNN
@@
 F 4 "C25130" H 6650 3175 50  0001 C CNN "LCSC"
 F 5 "Chip Resistor - Surface Mount 680Ohms ±1% 1/16W 0402 RoHS" H 6650 3175 50  0001 C CNN "Desc"
+F 6 "0402WGF6800TCE" H 6650 3175 50  0001 C CNN "MPN"
 	1    6650 3175
 	-1   0    0    1
@@
 Connection ~ 5950 1475
 $Comp
-L Connector_Generic:Conn_02x03_Odd_Even J5
+L Connector_Generic:Conn_02x04_Odd_Even J5
 U 1 1 5F880CAC
 P 4475 1475
 F 0 "J5" H 4525 1800 50  0000 C CNN
 F 1 "PowerTP" H 4525 1700 50  0000 C CNN
-F 2 "Connector_PinHeader_2.54mm:PinHeader_2x03_P2.54mm_Vertical" H 4475 1475 50  0001 C CNN
+F 2 "Connector_PinHeader_2.54mm:PinHeader_2x04_P2.54mm_Vertical" H 4475 1475 50  0001 C CNN
 F 3 "~" H 4475 1475 50  0001 C CNN
+F 4 "DNP" H 4475 1475 50  0001 C CNN "MPN"
 	1    4475 1475
 	1    0    0    -1
@@
 L power:GND #PWR0134
 U 1 1 5F881803
-P 4275 1575
-F 0 "#PWR0134" H 4275 1325 50  0001 C CNN
-F 1 "GND" H 4280 1402 50  0000 C CNN
-F 2 "" H 4275 1575 50  0001 C CNN
-F 3 "" H 4275 1575 50  0001 C CNN
-	1    4275 1575
+P 4275 1675
+F 0 "#PWR0134" H 4275 1425 50  0001 C CNN
+F 1 "GND" H 4280 1502 50  0000 C CNN
+F 2 "" H 4275 1675 50  0001 C CNN
+F 3 "" H 4275 1675 50  0001 C CNN
+	1    4275 1675
 	1    0    0    -1
 $EndComp
@@
 F 2 "Capacitor_SMD:C_0402_1005Metric" H 2175 3225 50  0001 C CNN
 F 3 "" H 2175 3225 50  0001 C CNN
-F 4 "CC0402KRX5R6BB105" H 2205 3375 20  0001 C CNN "MPN"
-F 5 "302010040" H 2205 3375 20  0001 C CNN "SKU"
-F 6 "C52923" H 2175 3225 50  0001 C CNN "LCSC"
+F 4 "CL05A105KA5NQNC" H 2205 3375 20  0001 C CNN "MPN"
+F 5 "C52923" H 2175 3225 50  0001 C CNN "LCSC"
 	1    2175 3225
 	-1   0    0    -1
@@
 F 5 "C134819-DNP" H 1600 3275 50  0001 C CNN "LCSC"
 F 6 " " H 1600 3275 50  0001 C CNN "SKU"
+F 7 "https://lcsc.com/product-detail/Aluminum-Electrolytic-Capacitors-SMD_Lelon-VZH221M1HTR-1010_C134819.html/?href=jlc-SMT" H 1600 3275 50  0001 C CNN "Link"
+F 8 "LCSC" H 1600 3275 50  0001 C CNN "Vendor"
 	1    1600 3275
 	1    0    0    -1
@@
 F 3 "~" H 4325 6700 50  0001 C CNN
 F 4 "C25798" H 4325 6700 50  0001 C CNN "LCSC"
+F 5 "0402WGF7502TCE" H 4325 6700 50  0001 C CNN "MPN"
 	1    4325 6700
 	1    0    0    -1
@@
 F 3 "~" H 4325 7050 50  0001 C CNN
 F 4 "C25778" H 4325 7050 50  0001 C CNN "LCSC"
+F 5 "0402WGF3303TCE" H 4325 7050 50  0001 C CNN "MPN"
 	1    4325 7050
 	-1   0    0    1
@@
 F 3 "" H 3250 6350 50  0001 C CNN
 F 4 "C15195" H 3250 6350 50  0001 C CNN "LCSC"
+F 5 "CL05B103KB5NNNC" H 3250 6350 50  0001 C CNN "MPN"
 	1    3250 6350
 	-1   0    0    1
@@
 	5150 950  3750 950
 $Bitmap
-Pos 1925 1050
+Pos 2000 1250
 Scale 0.700000
 Data
@@
 F 1 "2.2NF" H 3100 5125 45  0000 L CNN
 F 2 "Capacitor_SMD:C_0402_1005Metric" H 3350 5200 50  0001 C CNN
-F 3 "https://statics3.seeedstudio.com/images/opl/datasheet/302010022.pdf" H 3350 5200 50  0001 C CNN
-F 4 "CC0402KRX7R9BB222" H 3380 5350 20  0001 C CNN "MPN"
-F 5 "302010022" V 3434 5268 20  0001 L CNN "SKU"
-F 6 "C1531" H 3350 5200 50  0001 C CNN "LCSC"
+F 3 "" H 3350 5200 50  0001 C CNN
+F 4 "0402B222K500NT" H 3380 5350 20  0001 C CNN "MPN"
+F 5 "C1531" H 3350 5200 50  0001 C CNN "LCSC"
+F 6 "https://lcsc.com/product-detail/Multilayer-Ceramic-Capacitors-MLCC-SMD-SMT_2-2nF-222-10-50V_C1531.html/?href=jlc-SMT" H 3350 5200 50  0001 C CNN "Link"
+F 7 "LCSC" H 3350 5200 50  0001 C CNN "Vendor"
 	1    3350 5200
 	-1   0    0    -1
@@
 F 2 "TestPoint:TestPoint_Pad_D2.0mm" H 5700 4900 50  0001 C CNN
 F 3 "~" H 5700 4900 50  0001 C CNN
+F 4 "DNP" H 5500 4900 50  0001 C CNN "MPN"
 	1    5500 4900
 	0    1    1    0
@@
 F 2 "TestPoint:TestPoint_Pad_D2.0mm" H 4900 6550 50  0001 C CNN
 F 3 "~" H 4900 6550 50  0001 C CNN
+F 4 "DNP" H 4700 6550 50  0001 C CNN "MPN"
 	1    4700 6550
 	0    1    1    0
 $EndComp
-$Comp
-L Connector_Generic:Conn_01x02 J12
-U 1 1 5F510E13
-P 4575 1850
-F 0 "J12" H 4655 1842 50  0000 L CNN
-F 1 "GND" H 4655 1751 50  0000 L CNN
-F 2 "Connector_PinHeader_2.54mm:PinHeader_1x02_P2.54mm_Vertical" H 4575 1850 50  0001 C CNN
-F 3 "~" H 4575 1850 50  0001 C CNN
-	1    4575 1850
-	1    0    0    -1
-$EndComp
-$Comp
-L power:GND #PWR0165
-U 1 1 5F511940
-P 4375 1950
-F 0 "#PWR0165" H 4375 1700 50  0001 C CNN
-F 1 "GND" H 4225 1875 50  0000 C CNN
-F 2 "" H 4375 1950 50  0001 C CNN
-F 3 "" H 4375 1950 50  0001 C CNN
-	1    4375 1950
-	1    0    0    -1
-$EndComp
-Wire Wire Line
-	4375 1850 4375 1950
-Connection ~ 4375 1950
 Wire Notes Line
 	5150 950  5150 2125
@@
 F 2 "Capacitor_SMD:C_0402_1005Metric" H 4525 3425 50  0001 C CNN
 F 3 "" H 4525 3425 50  0001 C CNN
-F 4 "CC0402KRX5R6BB105" H 4555 3575 20  0001 C CNN "MPN"
-F 5 "302010040" H 4555 3575 20  0001 C CNN "SKU"
-F 6 "C52923" H 4525 3425 50  0001 C CNN "LCSC"
+F 4 "CL05A105KA5NQNC" H 4555 3575 20  0001 C CNN "MPN"
+F 5 "C52923" H 4525 3425 50  0001 C CNN "LCSC"
 	1    4525 3425
 	-1   0    0    -1
@@
 Wire Wire Line
 	1650 6200 1650 6350
+Wire Wire Line
+	4275 1575 4275 1675
+Connection ~ 4275 1675
+Text GLabel 4775 1675 2    51   Input ~ 0
+PGND
 $EndSCHEMATC
