File: mark-II-Rpi-devkit/KiCAD/SJ201-Raspberry Pi 4 Daughterboard/Power.sch (KiCad schematic (older format))
At the start: 41 parts, among them J1 Barrel_Jack, J5 PowerTP, J8 PWR, Q3 AO3401A, U1 XL4501E1, U12 TPS75933KTTR, U15 AMS1117-1.8, U4 AMS1117-3.3, U7 MP2359

Commit message: Updated files for R6 v2
Parts:
- C66: value 1uF -> 1uF-DNP; LCSC C7174 -> C7174-DNP; MPN TAJA105K016RNJ -> TAJA105K016RNJ-DNP
- C67: value 470uF -> 470uF-DNP; LCSC C79114 -> C79114-DNP; MPN 6TPE470MAZU -> 6TPE470MAZU-DNP
- C68: value 10UF -> 10uF-DNP; LCSC C15525 -> C15525-DNP; MPN CC0402MRX5R5BB106 -> CC0402MRX5R5BB106-DNP; SKU 302010053 -> 302010053-DNP
- C69: value 22UF -> 22UF-DNP; LCSC C59461 -> C59461-DNP; MPN CL10A226MQ8NRNE -> CL10A226MQ8NRNE-DNP
- R51: value 3.3K -> 3.3K-DNP; LCSC C25890 -> C25890-DNP; MPN 0402WGF3301TCE -> 0402WGF3301TCE-DNP
- U12: value TPS75933KTTR -> TPS75933KTTR-DNP; MPN TPS75933KTTR -> TPS75933KTTR-DNP
- U15: value AMS1117-1.8 -> AMS1117-1.8-DNP; LCSC C6185 -> C6185-DNP; MPN AMS1117-1.8 -> AMS1117-1.8-DNP
- U4: MPN AMS1117-3.3-DNP -> AMS1117-3.3
Changed lines of the file:
@@
 Sheet 2 8
 Title "Power"
-Date "2020-12-30"
-Rev "Rev5 - v1"
+Date "2021-01-27"
+Rev "Rev6 - v2"
 Comp "Mycroft AI"
 Comment1 "SJ-201-R6"
@@
 F 4 "C6186" H 1925 4750 50  0001 C CNN "LCSC"
 F 5 "https://lcsc.com/product-detail/Dropout-Regulators-LDO_ON-Semiconductor-ON-NCP565ST12T3G_C556400.html" H 1925 4750 50  0001 C CNN "Link"
-F 6 "AMS1117-3.3-DNP" H 1925 4750 50  0001 C CNN "MPN"
+F 6 "AMS1117-3.3" H 1925 4750 50  0001 C CNN "MPN"
 	1    1925 4750
 	1    0    0    -1
@@
 P 4550 4875
 F 0 "U12" H 4550 5217 50  0000 C CNN
-F 1 "TPS75933KTTR" H 4550 5126 50  0000 C CNN
+F 1 "TPS75933KTTR-DNP" H 4550 5126 50  0000 C CNN
 F 2 "Package_TO_SOT_SMD:TO-263-5_TabPin3" H 4550 4875 50  0001 C CNN
 F 3 "https://www.ti.com/lit/ds/slvs318e/slvs318e.pdf" H 4550 4875 50  0001 C CNN
 F 4 "https://www.digikey.com/en/products/detail/texas-instruments/TPS75933KTTR/1673190" H 4550 4875 50  0001 C CNN "Digikey"
-F 5 "TPS75933KTTR" H 4550 4875 50  0001 C CNN "MPN"
+F 5 "TPS75933KTTR-DNP" H 4550 4875 50  0001 C CNN "MPN"
 F 6 "https://www.digikey.com/en/products/detail/texas-instruments/TPS75933KTTR/1673190" H 4550 4875 50  0001 C CNN "Link"
 	1    4550 4875
@@
 P 3800 4950
 F 0 "C66" H 3891 4996 50  0000 L CNN
-F 1 "1uF" H 3891 4905 50  0000 L CNN
+F 1 "1uF-DNP" H 3800 4850 50  0000 L CNN
 F 2 "Capacitor_Tantalum_SMD:CP_EIA-3216-10_Kemet-I" H 3800 4950 50  0001 C CNN
 F 3 "~" H 3800 4950 50  0001 C CNN
-F 4 "TAJA105K016RNJ" H 3800 4950 50  0001 C CNN "MPN"
-F 5 "C7174" H 3800 4950 50  0001 C CNN "LCSC"
+F 4 "TAJA105K016RNJ-DNP" H 3800 4950 50  0001 C CNN "MPN"
+F 5 "C7174-DNP" H 3800 4950 50  0001 C CNN "LCSC"
 F 6 "https://lcsc.com/product-detail/Tantalum-Capacitors_AVX-TAJA105K016RNJ_C7174.html" H 3800 4950 50  0001 C CNN "Link"
 	1    3800 4950
@@
 AR Path="/5EAAC9A5/5FA5481E" Ref="R51"  Part="1"
 F 0 "R51" H 5000 4850 50  0000 L CNN
-F 1 "3.3K" H 4975 4950 50  0000 L CNN
+F 1 "3.3K-DNP" H 4950 5050 50  0000 L CNN
 F 2 "Resistor_SMD:R_0402_1005Metric" H 5200 4875 50  0001 C CNN
 F 3 "~" H 5200 4875 50  0001 C CNN
-F 4 "0402WGF3301TCE" H 5200 4875 50  0001 C CNN "MPN"
-F 5 "C25890" H 5200 4875 50  0001 C CNN "LCSC"
+F 4 "0402WGF3301TCE-DNP" H 5200 4875 50  0001 C CNN "MPN"
+F 5 "C25890-DNP" H 5200 4875 50  0001 C CNN "LCSC"
 F 6 "RC0402FR-073K3L" H 5200 4875 50  0001 C CNN "Tempo"
 	1    5200 4875
@@
 P 5700 4950
 F 0 "C67" H 5750 5075 45  0000 L CNN
-F 1 "470uF " H 5750 4825 45  0000 L CNN
+F 1 "470uF-DNP" H 5750 4825 45  0000 L CNN
 F 2 "Capacitor_Tantalum_SMD:CP_EIA-7343-15_Kemet-W" H 5700 4950 50  0001 C CNN
 F 3 "" H 5700 4950 50  0001 C CNN
-F 4 "6TPE470MAZU" H 5730 5100 20  0001 C CNN "MPN"
-F 5 "C79114" H 5700 4950 50  0001 C CNN "LCSC"
+F 4 "6TPE470MAZU-DNP" H 5730 5100 20  0001 C CNN "MPN"
+F 5 "C79114-DNP" H 5700 4950 50  0001 C CNN "LCSC"
 F 6 " " H 5700 4950 50  0001 C CNN "SKU"
 F 7 "LCSC" H 5700 4950 50  0001 C CNN "Vendor"
@@
 	3600 4300 6425 4300
 $Comp
-L Regulator_Linear:AMS1117-1.8 U15
-U 1 1 5FFE9528
-P 7375 4775
-F 0 "U15" H 7375 5017 50  0000 C CNN
-F 1 "AMS1117-1.8" H 7375 4926 50  0000 C CNN
-F 2 "Package_TO_SOT_SMD:SOT-223-3_TabPin2" H 7375 4975 50  0001 C CNN
-F 3 "http://www.advanced-monolithic.com/pdf/ds1117.pdf" H 7475 4525 50  0001 C CNN
-F 4 "C6185" H 7375 4775 50  0001 C CNN "LCSC"
-F 5 "AMS1117-1.8" H 7375 4775 50  0001 C CNN "MPN"
-F 6 "https://lcsc.com/product-detail/Dropout-Regulators-LDO_Advanced-Monolithic-Systems-AMS1117-1-8_C6185.html" H 7375 4775 50  0001 C CNN "Link"
-	1    7375 4775
-	1    0    0    -1
-$EndComp
-$Comp
-L Device:C_Small C?
-U 1 1 5FFEA269
-P 6900 4925
-AR Path="/5EA9C76D/5FFEA269" Ref="C?"  Part="1"
-AR Path="/5EA9C461/5FFEA269" Ref="C?"  Part="1"
-AR Path="/5EAAC9A5/5FFEA269" Ref="C68"  Part="1"
-F 0 "C68" H 7100 4975 45  0000 R CNN
-F 1 "10UF" H 7125 4850 45  0000 R CNN
-F 2 "Capacitor_SMD:C_0402_1005Metric" H 6900 4925 50  0001 C CNN
-F 3 "" H 6900 4925 50  0001 C CNN
-F 4 "CC0402MRX5R5BB106" H 6930 5075 20  0001 C CNN "MPN"
-F 5 "302010053" V 6816 4857 20  0001 R CNN "SKU"
-F 6 "C15525" H 6900 4925 50  0001 C CNN "LCSC"
-	1    6900 4925
-	1    0    0    -1
-$EndComp
-$Comp
 L power:+5V #PWR0141
 U 1 1 5FFEA5EF
@@
 $EndComp
 $Comp
-L Device:C_Small C?
-U 1 1 5FFEB13B
-P 7800 4925
-AR Path="/5EA9C76D/5FFEB13B" Ref="C?"  Part="1"
-AR Path="/5EA9C461/5FFEB13B" Ref="C?"  Part="1"
-AR Path="/5EAAC9A5/5FFEB13B" Ref="C69"  Part="1"
-F 0 "C69" H 7975 5000 45  0000 R CNN
-F 1 "22UF" H 8025 4850 45  0000 R CNN
-F 2 "Capacitor_SMD:C_0603_1608Metric" H 7800 4925 50  0001 C CNN
-F 3 "" H 7800 4925 50  0001 C CNN
-F 4 "CL10A226MQ8NRNE" H 7800 4925 50  0001 C CNN "MPN"
-F 5 "C59461" H 7800 4925 50  0001 C CNN "LCSC"
-	1    7800 4925
-	1    0    0    -1
-$EndComp
-$Comp
 L power:+1V8 #PWR0196
 U 1 1 5FFEBCD6
@@
 	1    0    0    -1
 $EndComp
+$Comp
+L Regulator_Linear:AMS1117-1.8 U15
+U 1 1 5FFE9528
+P 7375 4775
+F 0 "U15" H 7375 5017 50  0000 C CNN
+F 1 "AMS1117-1.8-DNP" H 7300 4925 50  0000 C CNN
+F 2 "Package_TO_SOT_SMD:SOT-223-3_TabPin2" H 7375 4975 50  0001 C CNN
+F 3 "http://www.advanced-monolithic.com/pdf/ds1117.pdf" H 7475 4525 50  0001 C CNN
+F 4 "C6185-DNP" H 7375 4775 50  0001 C CNN "LCSC"
+F 5 "AMS1117-1.8-DNP" H 7375 4775 50  0001 C CNN "MPN"
+F 6 "https://lcsc.com/product-detail/Dropout-Regulators-LDO_Advanced-Monolithic-Systems-AMS1117-1-8_C6185.html" H 7375 4775 50  0001 C CNN "Link"
+	1    7375 4775
+	1    0    0    -1
+$EndComp
+$Comp
+L Device:C_Small C?
+U 1 1 5FFEA269
+P 6900 4925
+AR Path="/5EA9C76D/5FFEA269" Ref="C?"  Part="1"
+AR Path="/5EA9C461/5FFEA269" Ref="C?"  Part="1"
+AR Path="/5EAAC9A5/5FFEA269" Ref="C68"  Part="1"
+F 0 "C68" H 7100 4975 45  0000 R CNN
+F 1 "10uF-DNP" H 7075 4850 45  0000 R CNN
+F 2 "Capacitor_SMD:C_0402_1005Metric" H 6900 4925 50  0001 C CNN
+F 3 "" H 6900 4925 50  0001 C CNN
+F 4 "CC0402MRX5R5BB106-DNP" H 6930 5075 20  0001 C CNN "MPN"
+F 5 "302010053-DNP" V 6816 4857 20  0001 R CNN "SKU"
+F 6 "C15525-DNP" H 6900 4925 50  0001 C CNN "LCSC"
+	1    6900 4925
+	1    0    0    -1
+$EndComp
+$Comp
+L Device:C_Small C?
+U 1 1 5FFEB13B
+P 7800 4925
+AR Path="/5EA9C76D/5FFEB13B" Ref="C?"  Part="1"
+AR Path="/5EA9C461/5FFEB13B" Ref="C?"  Part="1"
+AR Path="/5EAAC9A5/5FFEB13B" Ref="C69"  Part="1"
+F 0 "C69" H 7975 5000 45  0000 R CNN
+F 1 "22UF-DNP" H 7975 4850 45  0000 R CNN
+F 2 "Capacitor_SMD:C_0603_1608Metric" H 7800 4925 50  0001 C CNN
+F 3 "" H 7800 4925 50  0001 C CNN
+F 4 "CL10A226MQ8NRNE-DNP" H 7800 4925 50  0001 C CNN "MPN"
+F 5 "C59461-DNP" H 7800 4925 50  0001 C CNN "LCSC"
+	1    7800 4925
+	1    0    0    -1
+$EndComp

Commit message: Update libraries, reorganize files
Parts:
- FB8: symbol kevin:Ferrite_Bead_Small -> Mycroft:Ferrite_Bead_Small
- U1: symbol user:XL4015 -> Mycroft:XL4015
- U12: symbol user:TPS759xxx -> Mycroft:TPS759xxx
- U7: symbol user:MP2359 -> Mycroft:MP2359
Changed lines of the file:
@@
 Connection ~ 1475 4750
 $Comp
-L kevin:Ferrite_Bead_Small L?
+L Mycroft:Ferrite_Bead_Small L?
 U 1 1 5F089568
 P 8350 1175
@@
 AR Path="/5EA9C67D/5F089568" Ref="L?"  Part="1"
 AR Path="/5EAAC9A5/5F089568" Ref="FB8"  Part="1"
+AR Path="/5F089568" Ref="FB8"  Part="1"
 F 0 "FB8" V 8300 1075 50  0000 C CNN
 F 1 "FB" V 8300 1325 50  0000 C CNN
@@
 	3550 2000 3550 475
 $Comp
-L user:XL4015 U1
-U 1 1 5F0C10B6
-P 3225 3175
-F 0 "U1" H 3250 3543 51  0000 C CNN
-F 1 "XL4501E1" H 3250 3450 51  0000 C CNN
-F 2 "Package_TO_SOT_SMD:TO-263-5_TabPin3" H 3225 3175 51  0001 C CNN
-F 3 "https://datasheet.lcsc.com/szlcsc/2001091809_XLSEMI-XL4501E1_C73025.pdf" H 3225 3175 51  0001 C CNN
-F 4 "XL4501E1" H 3225 3175 50  0001 C CNN "MPN"
-F 5 "C73025" H 3225 3175 50  0001 C CNN "LCSC"
-F 6 "https://lcsc.com/product-detail/DC-DC-Converters_XLSEMI-XL4501E1_C73025.html" H 3225 3175 50  0001 C CNN "Link"
-	1    3225 3175
-	1    0    0    -1
-$EndComp
-$Comp
 L Device:R_Small R?
 U 1 1 5F0CD0DA
@@
 	-1   0    0    1
 $EndComp
-$Comp
-L user:MP2359 U?
-U 1 1 5F44B3BE
-P 2700 6350
-AR Path="/5EA9C76D/5F44B3BE" Ref="U?"  Part="1"
-AR Path="/5EAAC9A5/5F44B3BE" Ref="U7"  Part="1"
-F 0 "U7" H 2500 6650 63  0000 C CNN
-F 1 "MP2359" H 2400 5775 45  0000 C CNN
-F 2 "Package_TO_SOT_SMD:TSOT-23-6" H 2700 6350 63  0001 C CNN
-F 3 "https://www.monolithicpower.com/en/documentview/productdocument/index/version/2/document_type/Datasheet/lang/en/sku/MP2359/document_id/228" H 2700 6350 63  0001 C CNN
-F 4 "MP2359DJ-LF-Z" H 2700 6350 50  0001 C CNN "MPN"
-F 5 "https://www.mouser.com/ProductDetail/Monolithic-Power-Systems-MPS/MP2359DJ-LF-Z/?qs=rC7bBWoQAAkgAaURxgQSyA%3D%3D" H 2700 6350 50  0001 C CNN "Link"
-F 6 "C14259" H 2700 6350 50  0001 C CNN "LCSC"
-	1    2700 6350
-	1    0    0    -1
-$EndComp
 Wire Wire Line
 	3150 6200 3250 6200
@@
 	1100 4300 3325 4300
 $Comp
-L user:TPS759xxx U12
+L Mycroft:TPS759xxx U12
 U 1 1 5FCCB82B
 P 4550 4875
+AR Path="/5FCCB82B" Ref="U12"  Part="1"
+AR Path="/5EAAC9A5/5FCCB82B" Ref="U12"  Part="1"
 F 0 "U12" H 4550 5217 50  0000 C CNN
 F 1 "TPS75933KTTR-DNP" H 4550 5126 50  0000 C CNN
@@
 	1    0    0    -1
 $EndComp
+$Comp
+L Mycroft:MP2359 U?
+U 1 1 5F44B3BE
+P 2700 6350
+AR Path="/5EA9C76D/5F44B3BE" Ref="U?"  Part="1"
+AR Path="/5EAAC9A5/5F44B3BE" Ref="U7"  Part="1"
+AR Path="/5F44B3BE" Ref="U7"  Part="1"
+F 0 "U7" H 2500 6650 63  0000 C CNN
+F 1 "MP2359" H 2400 5775 45  0000 C CNN
+F 2 "Package_TO_SOT_SMD:TSOT-23-6" H 2700 6350 63  0001 C CNN
+F 3 "https://www.monolithicpower.com/en/documentview/productdocument/index/version/2/document_type/Datasheet/lang/en/sku/MP2359/document_id/228" H 2700 6350 63  0001 C CNN
+F 4 "MP2359DJ-LF-Z" H 2700 6350 50  0001 C CNN "MPN"
+F 5 "https://www.mouser.com/ProductDetail/Monolithic-Power-Systems-MPS/MP2359DJ-LF-Z/?qs=rC7bBWoQAAkgAaURxgQSyA%3D%3D" H 2700 6350 50  0001 C CNN "Link"
+F 6 "C14259" H 2700 6350 50  0001 C CNN "LCSC"
+	1    2700 6350
+	1    0    0    -1
+$EndComp
+$Comp
+L Mycroft:XL4015 U1
+U 1 1 5F0C10B6
+P 3225 3175
+AR Path="/5F0C10B6" Ref="U1"  Part="1"
+AR Path="/5EAAC9A5/5F0C10B6" Ref="U1"  Part="1"
+F 0 "U1" H 3250 3543 51  0000 C CNN
+F 1 "XL4501E1" H 3250 3450 51  0000 C CNN
+F 2 "Package_TO_SOT_SMD:TO-263-5_TabPin3" H 3225 3175 51  0001 C CNN
+F 3 "https://datasheet.lcsc.com/szlcsc/2001091809_XLSEMI-XL4501E1_C73025.pdf" H 3225 3175 51  0001 C CNN
+F 4 "XL4501E1" H 3225 3175 50  0001 C CNN "MPN"
+F 5 "C73025" H 3225 3175 50  0001 C CNN "LCSC"
+F 6 "https://lcsc.com/product-detail/DC-DC-Converters_XLSEMI-XL4501E1_C73025.html" H 3225 3175 50  0001 C CNN "Link"
+	1    3225 3175
+	1    0    0    -1
+$EndComp
