File: mark-II-Rpi-devkit/KiCAD/SJ201-Raspberry Pi 4 Daughterboard/MCU.sch (KiCad schematic (older format))
At the start: 22 parts, among them J10 Conn_01x04, J7 FanConnector, Q1 MMBT3904, Q2 BSS138, Q4 BSS138, Q5 BSS138, Q6 BSS138, U13 ATtiny1614-SS

Commit message: Updated files for R6 v2
Parts:
- Q2, Q4, Q5, Q6: value BSS138 -> BSS138-DNP; LCSC C112239 -> C112239-DNP; MPN BSS138 -> BSS138-DNP
- R29, R37, R55, R56, R58, R59: value 10k -> 10k-DNP; LCSC C25744 -> C25744-DNP; MPN RC0402FR-0710KL -> RC0402FR-0710KL-DNP
- R54: value 10k -> 10k-DNP
- R60: value 10k -> 10k-DNP; MPN RC0402FR-0710KL -> RC0402FR-0710KL-DNP

Commit message: Removed unused files, cleaned up directory, remove SJ202
Parts:
- J7: footprint user:FanPinHeader_1x04_P2.54mm_Vertical -> Mycroft:FanPinHeader_1x04_P2.54mm_Vertical
Changed lines of the file:
@@
 F 0 "J7" H 3868 5700 50  0000 C CNN
 F 1 "FanConnector" H 3868 5791 50  0000 C CNN
-F 2 "user:FanPinHeader_1x04_P2.54mm_Vertical" H 3950 6125 50  0001 C CNN
+F 2 "Mycroft:FanPinHeader_1x04_P2.54mm_Vertical" H 3950 6125 50  0001 C CNN
 F 3 "~" H 3950 6125 50  0001 C CNN
 F 4 "744-81-04TG1B" H 3950 6125 50  0001 C CNN "MPN"
