File: mark-II-Rpi-devkit/KiCAD/SJ201-Raspberry Pi 4 Daughterboard/SJ-201-R6.sch (KiCad schematic (older format))
At the start: 8 parts

Commit message: Update libraries, reorganize files
Parts:
- H5: footprint mycroft:mycroft_logo_graphic -> Logos:mycroft_logo_graphic
- H6: footprint libraries:simon-jestor-logo -> Logos:simon-jester-logo
- H7: footprint mycroft:mycroft_logo_words -> Logos:mycroft_logo_words
Changed lines of the file:
@@
 F 0 "H5" H 9250 6696 50  0001 L CNN
 F 1 "MountingHole" H 9250 6605 50  0001 L CNN
-F 2 "mycroft:mycroft_logo_graphic" H 9150 6650 50  0001 C CNN
+F 2 "Logos:mycroft_logo_graphic" H 9150 6650 50  0001 C CNN
 F 3 "~" H 9150 6650 50  0001 C CNN
 F 4 "DNP" H 9150 6650 50  0001 C CNN "MPN"
@@
 F 0 "H7" H 9425 6696 50  0001 L CNN
 F 1 "MountingHole" H 9425 6605 50  0001 L CNN
-F 2 "mycroft:mycroft_logo_words" H 9325 6650 50  0001 C CNN
+F 2 "Logos:mycroft_logo_words" H 9325 6650 50  0001 C CNN
 F 3 "~" H 9325 6650 50  0001 C CNN
 F 4 "DNP" H 9325 6650 50  0001 C CNN "MPN"
@@
 F 0 "H6" H 9225 6496 50  0001 L CNN
 F 1 "MountingHole" H 9225 6405 50  0001 L CNN
-F 2 "libraries:simon-jestor-logo" H 9125 6450 50  0001 C CNN
+F 2 "Logos:simon-jester-logo" H 9125 6450 50  0001 C CNN
 F 3 "~" H 9125 6450 50  0001 C CNN
 F 4 "DNP" H 9125 6450 50  0001 C CNN "MPN"
